File: original/variklio_valdiklis_orig.sch (KiCad schematic (older format))
At the start: 125 parts, among them J1 Conn_01x05, P1 Conn_01x01, P2 Conn_01x01, P3 Conn_01x01, Q200 IRF830, Q201 2N4401, Q202 2N3906, Q300 2N3906, Q801 IRF830, Q802 IRF830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

Commit message: schemos ir pcb paruosimas
Parts:
- C100, C101, C102: value CP -> 120x400V
- C200, C205: value C -> 102
- C201: value CP -> 220x25V
- C300: value CP -> 1.0x50V
- C600, C602, C603: value C -> 104
- C601: value C -> 10n; footprint (none) -> Capacitor_THT:C_Rect_L7.2mm_W3.0mm_P5.00mm_FKS2_FKP2_MKS2_MKP2
- C604: value C -> 473
- C605: value C -> 22n
- C606, C607, C608, C801, C811: value C -> 222
- C609: value CP -> 100x16V
- C800, C810, C820: value CP -> 33x25V
- C821: renamed from C21; value C -> 222
- TR1: value R -> SL12
- U600: symbol ics:MC33035 -> variklio_valdiklis_orig-rescue:MC33035-ics
- U602: symbol ics:MC33039 -> variklio_valdiklis_orig-rescue:MC33039-ics
- U800, U810: symbol ics:Si9910 -> variklio_valdiklis_orig-rescue:Si9910-ics
- U820: renamed from U20; symbol ics:Si9910 -> variklio_valdiklis_orig-rescue:Si9910-ics
Connections:
- wire segments 467 -> 466
Other:
- moved on the sheet: C101, C102, D?, U601A, U601C, U601D

Commit message: schemos ir plokstes analize
Parts:
- H600, H601, H602: symbol Sensor_Magnetic:A1101ELHL -> variklio_valdiklis_orig-rescue:A1101ELHL-Sensor_Magnetic
Changed lines of the file:
@@
 EESchema Schematic File Version 4
 LIBS:variklio_valdiklis_orig-cache
-EELAYER 30 0
+EELAYER 29 0
 EELAYER END
 $Descr A3 16535 11693
@@
 EAI
 $Comp
-L Sensor_Magnetic:A1101ELHL H600
+L variklio_valdiklis_orig-rescue:A1101ELHL-Sensor_Magnetic H600
 U 1 1 5E96890E
 P 4800 3050
@@
 $EndComp
 $Comp
-L Sensor_Magnetic:A1101ELHL H601
+L variklio_valdiklis_orig-rescue:A1101ELHL-Sensor_Magnetic H601
 U 1 1 5E969E5B
 P 5650 3050
@@
 $EndComp
 $Comp
-L Sensor_Magnetic:A1101ELHL H602
+L variklio_valdiklis_orig-rescue:A1101ELHL-Sensor_Magnetic H602
 U 1 1 5E96A56F
 P 6400 3050
