File: original/variklio_valdiklis_orig.sch (KiCad schematic (older format))
At the start: 124 parts, among them J1 Conn_01x05, P1 Conn_01x01, P2 Conn_01x01, P3 Conn_01x01, Q200 IRF830, Q201 2N4401, Q202 2N3906, Q300 2N3906, Q801 IRF830, Q802 IRF830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

Commit message: schemos paruosimas
Parts:
- C700: value C -> 4n7
- R207: value 980R(?) -> 1k
- R702: value 5W -> 0.1*/5W
- R801, R811, R821: value 380R -> 390R
- R804, R814, R824: value 3.8k(?) -> 100R
- U600: footprint Package_DIP:DIP-24_W7.62mm -> Package_SO:SOIC-24W_7.5x15.4mm_P1.27mm
- U602: footprint Package_DIP:DIP-8_W7.62mm -> Package_SO:SOIC-8_3.9x4.9mm_P1.27mm
- renumbered D601 to D600, D600 to D601
Connections:
- net GND: now also TR2.2; no longer TR2.1
- net at R502.2, U500.3 (+): now also TR2.1; no longer TR2.2
Other:
- moved on the sheet: C606, C700, D801, D811, D821, P1, P2, P3, Q801, Q802, Q811, Q812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
