File: original/variklio_valdiklis_orig_1.sch (KiCad schematic (older format))
At the start: 124 parts, among them J1 Conn_01x05, P1 Conn_01x01, P2 Conn_01x01, P3 Conn_01x01, Q200 IRF830, Q201 2N4401, Q202 2N3906, Q300 2N3906, Q801 IRF830, Q802 IRF830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

Commit message: schemos ir pcb ruosimas
Parts:
- gave numbers to parts that had none: 1
- renumbered D103 to D107
Changed lines of the file:
@@
 $EndComp
 $Comp
-L Comparator:LM393 U?
+L Comparator:LM393 U500
 U 3 1 5D6B46CE
 P 10900 6300
-F 0 "U?" H 10858 6346 50  0001 L CNN
+F 0 "U500" H 10858 6346 50  0001 L CNN
 F 1 "LM393" H 10858 6300 50  0001 L CNN
 F 2 "" H 10900 6300 50  0001 C CNN
@@
 	4050 8500 4150 8500
 $Comp
-L Device:D D103
+L Device:D D107
 U 1 1 624ED292
 P 2450 8950
-F 0 "D103" H 2550 9050 50  0000 R CNN
+F 0 "D107" H 2550 9050 50  0000 R CNN
 F 1 "1N4005" H 2600 8850 50  0000 R CNN
 F 2 "Diode_THT:D_DO-41_SOD81_P10.16mm_Horizontal" H 2450 8950 50  0001 C CNN
