File: variklio_valdiklis.sch (KiCad schematic (older format))
At the start: 125 parts, among them J1 Conn_01x05, P1 Conn_01x01, P2 Conn_01x01, P3 Conn_01x01, Q200 IRF830, Q201 2N4401, Q202 2N3906, Q300 2N3906, Q801 IRF830, Q802 IRF830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

Commit message: schemos ir plokstes analize
Parts:
- H600, H601, H602: symbol Sensor_Magnetic:A1101ELHL -> variklio_valdiklis-rescue:A1101ELHL-Sensor_Magnetic
- U20, U800, U810: symbol ics:Si9910 -> variklio_valdiklis-rescue:Si9910-ics
- U600: symbol ics:MC33035 -> variklio_valdiklis-rescue:MC33035-ics
- U602: symbol ics:MC33039 -> variklio_valdiklis-rescue:MC33039-ics
Changed lines of the file:
@@
 EESchema Schematic File Version 4
 LIBS:variklio_valdiklis-cache
-EELAYER 30 0
+EELAYER 29 0
 EELAYER END
 $Descr A3 16535 11693
@@
 ~FAULT
 $Comp
-L ics:MC33035 U600
+L variklio_valdiklis-rescue:MC33035-ics U600
 U 1 1 5D733183
 P 7600 5600
@@
 	12300 2350 12150 2350
 $Comp
-L ics:Si9910 U810
+L variklio_valdiklis-rescue:Si9910-ics U810
 U 1 1 5D85649F
 P 12800 3300
@@
 	11700 2250 11700 2350
 $Comp
-L ics:Si9910 U20
+L variklio_valdiklis-rescue:Si9910-ics U20
 U 1 1 5D73DF53
 P 12800 1800
@@
 EAI
 $Comp
-L Sensor_Magnetic:A1101ELHL H600
+L variklio_valdiklis-rescue:A1101ELHL-Sensor_Magnetic H600
 U 1 1 5E96890E
 P 4800 3050
@@
 $EndComp
 $Comp
-L Sensor_Magnetic:A1101ELHL H601
+L variklio_valdiklis-rescue:A1101ELHL-Sensor_Magnetic H601
 U 1 1 5E969E5B
 P 5650 3050
@@
 $EndComp
 $Comp
-L Sensor_Magnetic:A1101ELHL H602
+L variklio_valdiklis-rescue:A1101ELHL-Sensor_Magnetic H602
 U 1 1 5E96A56F
 P 6400 3050
@@
 	12400 4750 12350 4750
 $Comp
-L ics:Si9910 U800
+L variklio_valdiklis-rescue:Si9910-ics U800
 U 1 1 5D856BAA
 P 12800 4850
@@
 	5550 2550 6300 2550
 $Comp
-L ics:MC33039 U602
+L variklio_valdiklis-rescue:MC33039-ics U602
 U 1 1 68D8E883
 P 5250 5000

Commit message: schemos paruosimas
Parts:
- removed C21, C606, C607, C608, C700, C801, C811: C, symbol Device:C
- removed C800, C810, C820: CP, symbol Device:CP
- removed D602, D? (x2): 1N5818, symbol Device:D
- removed D800, D810, D820: 1N4005, symbol Device:D
- removed D801, D811, D821: D, symbol Device:D
- removed R603, R607, R608: 1.8k, symbol Device:R
- removed R700, R701, R703, R800, R801, R802, R803, R804, R805, R810, R811, R812, R813, R814, R820, R821, R822, R823, R824: R, symbol Device:R
- removed R702: 5W, symbol Device:R
- removed U20, U800, U810: Si9910, Package_DIP:DIP-8_W7.62mm, symbol variklio_valdiklis-rescue:Si9910-ics
- removed U601: ILQ2, symbol Isolator:ILQ74
- removed Z800, Z810, Z820: D_Zener, symbol Device:D_Zener
- added C?: 10n, symbol Device:C
- added C? (x2): 1.0x400V, symbol Device:CP
- added C? (x4): C, symbol Device:C
- added D?: 15V/5W, symbol Device:D_Zener
- added D? (x2): MUR140, symbol Device:D
- added D? (x3): LL4148, Diode_SMD:D_MiniMELF, symbol Device:D
- added D? (x3): 1N4744, symbol Device:D_Zener
- added D? (x3): 1N5818, symbol Device:D
- added R? (x4): 18k, symbol Device:R
- added R? (x11): R, symbol Device:R
- added R? (x3): 1M, symbol Device:R
- added R?: 5W, symbol Device:R
- added U?: NE555, symbol Timer:NE555
- added U? (x3): MOC8204, Package_DIP:DIP-6_W7.62mm_SMDSocket_SmallPads, symbol Isolator:CNY17-4
- U600: footprint Package_DIP:DIP-24_W7.62mm -> Package_SO:SOIC-24W_7.5x15.4mm_P1.27mm
- U602: footprint Package_DIP:DIP-8_W7.62mm -> Package_SO:SOIC-8_3.9x4.9mm_P1.27mm
Connections:
- net labels added: AB, AT, BB, BT, CB, CT, ISENSE, OKM, OKP
- net labels removed: EAI, ~FAULT
- wire segments 467 -> 393
- no-connect marks 0 -> 2
Other:
- moved on the sheet: C300, C600, C601, C602, C603, C604, C605, C609, D300, H600, H601, H602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

Commit message: schemos ir pcb ruosimas
Parts:
- removed D100, D101, D102, D103: 1N5626, Diode_THT:D_DO-201_P15.24mm_Horizontal, symbol Device:D
- added D100: KBU8M, Diode_THT:Diode_Bridge_Vishay_KBU, symbol Diode_Bridge:KBU8M
- C100, C101, C102: value CP -> 120.0x400V
- C200, C205: value C -> 1nF; footprint (none) -> Capacitor_SMD:C_0805_2012Metric
- C300: value CP -> 1.0x50V
- C600, C602, C603: value C -> 0.1; footprint (none) -> Capacitor_SMD:C_0805_2012Metric
- C601: value C -> 10n; footprint (none) -> Capacitor_SMD:C_0805_2012Metric
- C604: value C -> 47n; footprint (none) -> Capacitor_SMD:C_0805_2012Metric
- C605: value C -> 22n; footprint (none) -> Capacitor_SMD:C_0805_2012Metric
- C606, C607, C608: renamed from C?; value C -> 2n2; footprint (none) -> Capacitor_SMD:C_0805_2012Metric
- C700: renamed from C?; value C -> 4n7; footprint (none) -> Capacitor_SMD:C_0805_2012Metric
- C801: renamed from C?; footprint (none) -> Capacitor_SMD:C_0805_2012Metric
- D103: value 1N4005 -> LL4005; footprint Diode_THT:D_DO-41_SOD81_P10.16mm_Horizontal -> Diode_SMD:D_MELF
- D104: value 1N4006 -> LL4006; footprint Diode_THT:D_DO-41_SOD81_P10.16mm_Horizontal -> Diode_SMD:D_MELF
- D105: value D -> LL4005; footprint (none) -> Diode_SMD:D_MELF
- D106: renamed from D?; value D -> 1N4148
- D300: value 1N4005 -> LL4005; footprint (none) -> Diode_SMD:D_MELF
- R100: value R -> 330k
- R200: renamed from R?; value R -> 180k
- R201, R204, R304, R602: value R -> 10k; footprint (none) -> Resistor_SMD:R_0805_2012Metric
- R202: value 47R -> 47R/5W
- R206, R305: value R -> 2.2k; footprint (none) -> Resistor_SMD:R_0805_2012Metric
- R207, R700, R701: renamed from R?; value R -> 1k; footprint (none) -> Resistor_SMD:R_0805_2012Metric
- R300: value R -> 1k; footprint (none) -> Resistor_SMD:R_0805_2012Metric
- R301: value R -> 490
- R302, R500, R502: value R -> 20k; footprint (none) -> Resistor_SMD:R_0805_2012Metric
- R303: value R -> 1M; footprint (none) -> Resistor_SMD:R_0805_2012Metric
- R306: value R -> 33k; footprint (none) -> Resistor_SMD:R_0805_2012Metric
- R307: value R -> 22k; footprint (none) -> Resistor_SMD:R_0805_2012Metric
- R501: value R -> 4.5k; footprint (none) -> Resistor_SMD:R_0805_2012Metric
- R600: value R -> 4.7k; footprint (none) -> Resistor_SMD:R_0805_2012Metric
- R601: renamed from R?; value R -> 150k; footprint (none) -> Resistor_SMD:R_0805_2012Metric
- R603, R607, R608: renamed from R?; value R -> 1.8k; footprint (none) -> Resistor_SMD:R_0805_2012Metric
- R605: value R -> 7.5k; footprint (none) -> Resistor_SMD:R_0805_2012Metric
- R606: value R -> 49k; footprint (none) -> Resistor_SMD:R_0805_2012Metric
- R702: renamed from R?; value 5W -> 0.1/2W
- R801, R805, R808, R811, R815, R821, R825: renamed from R?; footprint (none) -> Resistor_SMD:R_0805_2012Metric
- R803, R813, R823: renamed from R?; value R -> 72R; footprint (none) -> Resistor_SMD:R_0805_2012Metric
- R804, R814, R824: renamed from R?; value R -> 100R; footprint (none) -> Resistor_SMD:R_0805_2012Metric
- TR1: value R -> SL12
- Z200, Z201, Z203: renamed from ZD?; value D_Zener -> 1N5245
- gave numbers to parts that had none: 20
Connections:
- net ISENSE is gone; now on an unnamed net: C700.2, R700.2, R701.2
- net GND: now also U600.15 (~SENS)
- net at J1.4 (Pin_4): now also D100.2 (~~)
- net at C100.2, C101.2, C102.2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: now also D100.4 (-)
- net at Q821.1 (G), R821.2, U603.4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: now also R825.2; no longer R825.1
- net at P3.1 (Pin_1), Q821.3 (S), Q822.2 (D)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: now also R825.1; no longer R825.2
- net at Q811.1 (G), R811.2, U604.4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: now also R815.2; no longer R815.1
- net at P2.1 (Pin_1), Q811.3 (S), Q812.2 (D)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: now also R815.1; no longer R815.2
- net at Q801.1 (G), R801.2, U605.4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: now also R805.2; no longer R805.1
- net at P1.1 (Pin_1), Q801.3 (S), Q802.2 (D)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: now also R805.1; no longer R805.2
- net at D104.2 (A), F1.1: now also D100.3 (~~)
- net at TR1.2: now also D100.1 (+)
Other:
- moved on the sheet: C100, C101, C102, C600, C608, C700, D300, D602, D821, F1, P3, Q801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

Commit message: plokstes paruosimas, nauji pdf-ai
Parts:
- removed Q201: 2N4401, Package_TO_SOT_THT:TO-92_Inline, symbol Device:Q_NPN_EBC
- removed Q202, Q300: 2N3906, Package_TO_SOT_THT:TO-92_Inline, symbol Transistor_BJT:2N3906
- added C804, C805: 22x25V, Capacitor_THT:CP_Radial_D6.3mm_P2.50mm, symbol Device:CP
- added Q201: BC817, Package_TO_SOT_SMD:SOT-23, symbol Transistor_BJT:BC817
- added Q202, Q300: BC807, Package_TO_SOT_SMD:SOT-23, symbol Transistor_BJT:BC807
- added R100.1, R100.3: 100k, Resistor_SMD:R_1206_3216Metric, symbol Device:R_US
- C201: value CP -> 220x25V; footprint (none) -> Capacitor_THT:CP_Radial_D8.0mm_P2.50mm
- C300: footprint (none) -> Capacitor_THT:CP_Radial_D5.0mm_P2.50mm
- C609: value CP -> 100x16V; footprint (none) -> Capacitor_THT:CP_Radial_D5.0mm_P2.50mm
- C802: footprint (none) -> Capacitor_THT:CP_Radial_D10.0mm_P5.00mm
- C803: value 1.0x400V -> 22x25V; footprint (none) -> Capacitor_THT:CP_Radial_D6.3mm_P2.50mm
- D106: value 1N4148 -> LL4148; footprint (none) -> Diode_SMD:D_MiniMELF
- D600, D601, D602: footprint (none) -> Diode_SMD:D_SMA
- D805, D806: footprint (none) -> Diode_THT:D_DO-41_SOD81_P10.16mm_Horizontal
- F1: footprint (none) -> Fuse:Fuse_SunFuse-6HP
- H600, H601, H602: footprint (none) -> Connector_PinHeader_2.54mm:PinHeader_1x03_P2.54mm_Vertical
- J1: footprint (none) -> valdiklio_footprints:Jungtis
- P1, P2, P3: footprint (none) -> Connector_Pin:Pin_D1.0mm_L10.0mm
- Q200: footprint Package_TO_SOT_THT:TO-220-3_Vertical -> Package_TO_SOT_THT:TO-220-3_Horizontal_TabDown
- R100.2: renamed from R100; value 330k -> 100k; footprint (none) -> Resistor_SMD:R_1206_3216Metric
- R200: footprint (none) -> Resistor_THT:R_Axial_DIN0414_L11.9mm_D4.5mm_P15.24mm_Horizontal
- R202: footprint (none) -> Resistor_THT:R_Axial_Power_L25.0mm_W9.0mm_P30.48mm
- R301: footprint (none) -> Resistor_SMD:R_0805_2012Metric
- R604: value R -> 33k; footprint (none) -> Resistor_SMD:R_0805_2012Metric
- R702: footprint (none) -> Resistor_THT:R_Axial_DIN0411_L9.9mm_D3.6mm_P12.70mm_Horizontal
- TR1: footprint (none) -> Varistor:RV_Disc_D12mm_W3.9mm_P7.5mm
- U1: footprint (none) -> Package_DIP:DIP-6_W7.62mm
- U500, U606: footprint (none) -> Package_SO:SOIC-8_3.9x4.9mm_P1.27mm
- VP300: footprint (none) -> Potentiometer_THT:Potentiometer_ACP_CA6-H2,5_Horizontal
- Z200, Z201, Z203: footprint (none) -> Diode_THT:D_DO-35_SOD27_P7.62mm_Horizontal
- Z801, Z811, Z821: footprint (none) -> Diode_THT:D_DO-41_SOD81_P7.62mm_Horizontal
- Z804: value 15V/5W -> 1N5352; footprint (none) -> Diode_THT:D_DO-41_SOD81_P10.16mm_Horizontal
Connections:
- net +U: now also C804.2, C805.2
- net +V: now also R100.1.1; no longer R100.2.2
- net OKM: now also J1.5 (Pin_5); no longer J1.1 (Pin_1)
- net OKP: now also J1.4 (Pin_4); no longer J1.2 (Pin_2)
- net at R303.1, U1.4: now also Q300.2 (E)
- net at D100.2 (~~): now also J1.2 (Pin_2); no longer J1.4 (Pin_4)
- net at F1.2: now also J1.1 (Pin_1); no longer J1.5 (Pin_5)
- net at R302.2, R303.2, R304.1: now also Q300.1 (B)
- net at R305.1, R306.2: now also Q300.3 (C)
- net at C100.2, C101.2, C102.2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: now also Q201.2 (E), R100.3.1; no longer R100.2.1
- net at C803.1, D806.1 (K), U603.5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: now also C804.1, C805.1
- net at C205.1, R201.1, Z203.2 (A): now also Q202.2 (E)
- net at C200.2, R207.2: now also Q201.1 (B), Q202.3 (C)
- net at C205.2, R201.2: now also Q201.3 (C), Q202.1 (B)
- new net: R100.2.1, R100.3.2
- new net: R100.1.2, R100.2.2
Other:
- moved on the sheet: C600, C602, C603, R100.2, R200

Commit message: schemos ir plokstes paruosimas
Parts:
- added C610, C611, C612, C613: 0.1, Capacitor_SMD:C_0805_2012Metric, symbol Device:C
- added J2, J?: VB, TerminalBlock:TerminalBlock_bornier-2_P5.08mm, symbol Connector_Generic:Conn_01x02
- added J3, J4: IF, Connector_PinHeader_2.54mm:PinHeader_1x10_P2.54mm_Vertical, symbol Connector_Generic:Conn_01x10
- added J5, J6: HALLS, Connector_PinHeader_2.54mm:PinHeader_1x05_P2.54mm_Vertical, symbol Connector_Generic:Conn_01x05
- added J?: GND, Connector_PinHeader_2.54mm:PinHeader_1x04_P2.54mm_Vertical, symbol Connector_Generic:Conn_01x03
- H600: value HALL -> SA
- H601: value HALL -> SB
- H602: value HALL -> SC
Connections:
- net +U: now also J2.1 (Pin_1)
- net +V: now also J?.1 (Pin_1)
- net AB: now also J3.1 (Pin_1), J4.3 (Pin_3)
- net AT: now also J3.2 (Pin_2), J4.4 (Pin_4)
- net BB: now also J3.3 (Pin_3), J4.5 (Pin_5)
- net BT: now also J3.4 (Pin_4), J4.6 (Pin_6)
- net CB: now also J3.5 (Pin_5), J4.7 (Pin_7)
- net CT: now also J3.6 (Pin_6), J4.8 (Pin_8)
- net GND: now also C610.2, C611.1, C612.1, C613.1, J2.2 (Pin_2), J3.10 (Pin_10), J4.10 (Pin_10), J5.5 (Pin_5), J6.5 (Pin_5), J?.1 (Pin_1), J?.2 (Pin_2), J?.3 (Pin_3)
- net VCC: now also C610.1, C611.2, C612.2, C613.2, J4.1 (Pin_1), J4.2 (Pin_2), J5.1 (Pin_1), J6.1 (Pin_1)
- net at J1.1 (Pin_1): now also F1.1; no longer F1.2
- net ~SA: now reaches H600.2 (Vout), U600.4 (~SA), U602.1 (FC)
- net ~SA: now also J5.2 (Pin_2), J6.2 (Pin_2)
- net ~SB: now reaches H601.2 (Vout), U600.5 (~SB), U602.3 (FA)
- net ~SB: now also J5.3 (Pin_3), J6.3 (Pin_3)
- net ~SC: now reaches H602.2 (Vout), U600.6 (~SC), U602.2 (FB)
- net ~SC: now also J5.4 (Pin_4), J6.4 (Pin_4)
- net SENS: now reaches C700.2, R700.2, R701.2, U600.9 (SENS)
- net SENS: now also J3.9 (Pin_9), J4.9 (Pin_9)
- net at C100.2, C101.2, C102.2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: now also J?.2 (Pin_2)
- net at D100.3 (~~), D104.2 (A): now also F1.2; no longer F1.1
Other:
- moved on the sheet: C100, C101, C102, C200, C201, C205, C300, C600, C601, C602, C603, C604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
