File: variklio_valdiklis.kicad_pcb (KiCad board)
At the start: 2 copper layers, 134 x 134 mm, 18 parts

Commit message: schemos ir pcb paruosimas
Parts:
- removed >NAME (x5): >VALUE, SparkFun_Connectors:1X01_2MM
- added C100: CP_Radial_D22.0mm_P10.00mm_SnapIn, Capacitor_THT:CP_Radial_D22.0mm_P10.00mm_SnapIn, F.Cu at (51.0, 98.0)
- added C101: CP_Radial_D22.0mm_P10.00mm_SnapIn, Capacitor_THT:CP_Radial_D22.0mm_P10.00mm_SnapIn, F.Cu at (53.0, 74.0)
- added C102: CP_Radial_D22.0mm_P10.00mm_SnapIn, Capacitor_THT:CP_Radial_D22.0mm_P10.00mm_SnapIn, F.Cu at (65.0, 53.0)
- added F1: Fuseholder5x20_horiz_SemiClosed_Casing10x25mm, valdiklio_footprints:Fuseholder5x20_horiz_SemiClosed_Casing10x25mm, F.Cu at (91.0, 52.0)
- added J1: Jungtis, jungtis:Jungtis, F.Cu at (110.0, 30.0)
- added Q801: TO-220-3_Vertical, valdiklio_footprints:TO-220-3_Vertical, F.Cu at (84.7, 143.2)
- added Q802: TO-220-3_Vertical, valdiklio_footprints:TO-220-3_Vertical, F.Cu at (70.0, 133.0)
- added Q811: TO-220-3_Vertical, valdiklio_footprints:TO-220-3_Vertical, F.Cu at (121.8, 147.5)
- added Q812: TO-220-3_Vertical, valdiklio_footprints:TO-220-3_Vertical, F.Cu at (102.9, 148.5)
- added Q821: TO-220-3_Vertical, valdiklio_footprints:TO-220-3_Vertical, F.Cu at (139.7, 140.7)
- added Q822: TO-220-3_Vertical, valdiklio_footprints:TO-220-3_Vertical, F.Cu at (153.5, 129.8)
- turned REF** to 135 degrees

Commit message: schemos ir plokstes analize
Parts:
- added D100: Diode_Bridge_Vishay_KBU, Diode_THT:Diode_Bridge_Vishay_KBU, F.Cu at (85.0, 34.0)
- added D100: D_DO-201_P12.70mm_Horizontal, Diode_THT:D_DO-201_P12.70mm_Horizontal, F.Cu at (14.0, 29.9)
- added D101: D_DO-201_P12.70mm_Horizontal, Diode_THT:D_DO-201_P12.70mm_Horizontal, F.Cu at (19.9, 29.9)
- added D102: D_DO-201_P12.70mm_Horizontal, Diode_THT:D_DO-201_P12.70mm_Horizontal, F.Cu at (-2.00, 41.7)
- added D103: D_DO-201_P12.70mm_Horizontal, Diode_THT:D_DO-201_P12.70mm_Horizontal, F.Cu at (6.70, 44.3)
- moved F1 32.6 mm to (70.0, 27.0)
- moved C100 3.61 mm to (53.0, 101.0)
- moved C102 3.61 mm to (63.0, 56.0)
- moved C101 3.00 mm to (53.0, 77.0)

Commit message: schemos ir pcb ruosimas
Parts:
- removed the D100 at (14.0, 29.9)
- removed D101, D102, D103: D_DO-201_P12.70mm_Horizontal, Diode_THT:D_DO-201_P12.70mm_Horizontal
- removed F1: Fuseholder5x20_horiz_SemiClosed_Casing10x25mm, valdiklio_footprints:Fuseholder5x20_horiz_SemiClosed_Casing10x25mm
- C100, C101, C102: value CP_Radial_D22.0mm_P10.00mm_SnapIn -> 120x400V
- D100: value Diode_Bridge_Vishay_KBU -> 1N5626
- J1: value Jungtis -> Conn_01x05
- Q801, Q802, Q811, Q812, Q821, Q822: value TO-220-3_Vertical -> IRF830
- moved D100 8.94 mm to (77.0, 38.0)
Connections:
- C100 pad 1: (no net) -> /+V
- C100 pad 2: (no net) -> Net-(C100-Pad2)
- C101 pad 1: (no net) -> /+V
- C101 pad 2: (no net) -> Net-(C100-Pad2)
- C102 pad 1: (no net) -> /+V
- C102 pad 2: (no net) -> Net-(C100-Pad2)
- D100 pad 1: (no net) -> Net-(D100-Pad1)
- D100 pad 2: (no net) -> Net-(C100-Pad2)
- J1 pad 1: (no net) -> Net-(J1-Pad1)
- J1 pad 2: (no net) -> Net-(J1-Pad2)
- J1 pad 3: (no net) -> /PE
- J1 pad 4: (no net) -> Net-(D100-Pad1)
- J1 pad 5: (no net) -> Net-(F1-Pad2)
- Q801 pad 1: (no net) -> Net-(Q801-Pad1)
- Q801 pad 2: (no net) -> /+U
- Q801 pad 3: (no net) -> Net-(C800-Pad2)
- Q802 pad 1: (no net) -> Net-(D801-Pad2)
- Q802 pad 2: (no net) -> Net-(C800-Pad2)
- Q802 pad 3: (no net) -> Net-(Q802-Pad3)
- Q811 pad 1: (no net) -> Net-(Q811-Pad1)
- Q811 pad 2: (no net) -> /+U
- Q811 pad 3: (no net) -> Net-(C810-Pad2)
- Q812 pad 1: (no net) -> Net-(D811-Pad2)
- Q812 pad 2: (no net) -> Net-(C810-Pad2)
- Q812 pad 3: (no net) -> Net-(Q802-Pad3)
- Q821 pad 1: (no net) -> Net-(Q821-Pad1)
- Q821 pad 2: (no net) -> /+U
- Q821 pad 3: (no net) -> Net-(C820-Pad2)
- Q822 pad 1: (no net) -> Net-(D821-Pad2)
- Q822 pad 2: (no net) -> Net-(C820-Pad2)
- Q822 pad 3: (no net) -> Net-(Q802-Pad3)
Routing:
- added copper zone on B.Cu, net (none)

Commit message: schemos ir pcb ruosimas
Parts:
- added C200: 1nF, Capacitor_SMD:C_0805_2012Metric, F.Cu at (53.7, 14.0)
- added C205: 1nF, Capacitor_SMD:C_0805_2012Metric, F.Cu at (45.2, 23.2)
- added C600: 0.1, Capacitor_SMD:C_0805_2012Metric, F.Cu at (46.7, 17.3)
- added C601: 10n, Capacitor_SMD:C_0805_2012Metric, F.Cu at (58.4, 5.97)
- added C602: 0.1, Capacitor_SMD:C_0805_2012Metric, F.Cu at (40.8, 23.6)
- added C603: 0.1, Capacitor_SMD:C_0805_2012Metric, F.Cu at (45.2, 20.3)
- added C604: 47n, Capacitor_SMD:C_0805_2012Metric, F.Cu at (65.6, 0.18)
- added C605: 22n, Capacitor_SMD:C_0805_2012Metric, F.Cu at (49.3, 14.0)
- added C606: 2n2, Capacitor_SMD:C_0805_2012Metric, F.Cu at (71.7, 5.08)
- added C607: 2n2, Capacitor_SMD:C_0805_2012Metric, F.Cu at (53.7, 11.1)
- added C608: 2n2, Capacitor_SMD:C_0805_2012Metric, F.Cu at (73.3, -7.02)
- added C700: 4n7, Capacitor_SMD:C_0805_2012Metric, F.Cu at (49.3, 11.1)
- added C801: 10n, Capacitor_SMD:C_0805_2012Metric, F.Cu at (65.6, -2.77)
- added D103: LL4005, Diode_SMD:D_MELF, F.Cu at (88.0, -32.0)
- added D104: LL4006, Diode_SMD:D_MELF, F.Cu at (45.0, -34.0)
- added D105: LL4005, Diode_SMD:D_MELF, F.Cu at (45.0, -28.0)
- added D300: LL4005, Diode_SMD:D_MELF, F.Cu at (69.4, -22.0)
- added D801: LL4148, Diode_SMD:D_MiniMELF, F.Cu at (74.0, 130.2)
- added D811: LL4148, Diode_SMD:D_MiniMELF, F.Cu at (102.0, 139.0)
- added D821: LL4148, Diode_SMD:D_MiniMELF, F.Cu at (140.0, 133.0)
- added Q200: IRF830, Package_TO_SOT_THT:TO-220-3_Vertical, F.Cu at (95.5, -25.0)
- added Q201: 2N4401, Package_TO_SOT_THT:TO-92_Inline, F.Cu at (114.0, -26.0)
- added Q202: 2N3906, Package_TO_SOT_THT:TO-92_Inline, F.Cu at (106.5, -26.0)
- added Q300: 2N3906, Package_TO_SOT_THT:TO-92_Inline, F.Cu at (121.5, -26.0)
- added R201: 10k, Resistor_SMD:R_0805_2012Metric, F.Cu at (58.1, 8.92)
- added R204: 10k, Resistor_SMD:R_0805_2012Metric, F.Cu at (62.8, 6.08)
- added R206: 2.2k, Resistor_SMD:R_0805_2012Metric, F.Cu at (62.8, 3.13)
- added R207: 1k, Resistor_SMD:R_0805_2012Metric, F.Cu at (51.1, 17.0)
- added R300: 1k, Resistor_SMD:R_0805_2012Metric, F.Cu at (70.0, -0.82)
- added R302: 20k, Resistor_SMD:R_0805_2012Metric, F.Cu at (70.0, -3.77)
- added R303: 1M, Resistor_SMD:R_0805_2012Metric, F.Cu at (40.8, 20.6)
- added R304: 10k, Resistor_SMD:R_0805_2012Metric, F.Cu at (58.4, 3.02)
- added R305: 2.2k, Resistor_SMD:R_0805_2012Metric, F.Cu at (42.3, 17.3)
- added R306: 33k, Resistor_SMD:R_0805_2012Metric, F.Cu at (71.3, 9.03)
- added R307: 22k, Resistor_SMD:R_0805_2012Metric, F.Cu at (62.5, 14.9)
- added R500: 20k, Resistor_SMD:R_0805_2012Metric, F.Cu at (54.0, 22.9)
- added R501: 4.5k, Resistor_SMD:R_0805_2012Metric, F.Cu at (77.7, -7.02)
- added R502: 20k, Resistor_SMD:R_0805_2012Metric, F.Cu at (66.9, 9.03)
- added R600: 4.7k, Resistor_SMD:R_0805_2012Metric, F.Cu at (71.7, 2.13)
- added R601: 150k, Resistor_SMD:R_0805_2012Metric, F.Cu at (54.0, 19.9)
- added R602: 10k, Resistor_SMD:R_0805_2012Metric, F.Cu at (62.5, 12.0)
- added R603: 1.8k, Resistor_SMD:R_0805_2012Metric, F.Cu at (75.7, 8.03)
- added R605: 7.5k, Resistor_SMD:R_0805_2012Metric, F.Cu at (67.2, 6.08)
- added R606: 49k, Resistor_SMD:R_0805_2012Metric, F.Cu at (49.6, 23.2)
- added R607: 1.8k, Resistor_SMD:R_0805_2012Metric, F.Cu at (74.4, -1.12)
- added R608: 1.8k, Resistor_SMD:R_0805_2012Metric, F.Cu at (62.5, 9.03)
- added R700: 1k, Resistor_SMD:R_0805_2012Metric, F.Cu at (49.6, 20.3)
- added R701: 1k, Resistor_SMD:R_0805_2012Metric, F.Cu at (74.4, -4.07)
- added R801: 1M, Resistor_SMD:R_0805_2012Metric, F.Cu at (88.0, 117.0)
- added R803: 72R, Resistor_SMD:R_0805_2012Metric, F.Cu at (77.0, 131.1)
- added R804: 100R, Resistor_SMD:R_0805_2012Metric, F.Cu at (75.1, 126.0)
- added R805: 18k, Resistor_SMD:R_0805_2012Metric, F.Cu at (84.9, 130.0)
- added R808: 18k, Resistor_SMD:R_0805_2012Metric, F.Cu at (58.4, 23.8)
- added R811: 1M, Resistor_SMD:R_0805_2012Metric, F.Cu at (112.0, 128.0)
- added R813: 72R, Resistor_SMD:R_0805_2012Metric, F.Cu at (98.0, 142.0)
- added R814: 100R, Resistor_SMD:R_0805_2012Metric, F.Cu at (98.0, 138.0)
- added R815: 18k, Resistor_SMD:R_0805_2012Metric, F.Cu at (109.0, 141.0)
- added R821: 1M, Resistor_SMD:R_0805_2012Metric, F.Cu at (135.0, 117.0)
- added R823: 72R, Resistor_SMD:R_0805_2012Metric, F.Cu at (143.0, 134.0)
- added R824: 100R, Resistor_SMD:R_0805_2012Metric, F.Cu at (142.1, 129.0)
- added R825: 18k, Resistor_SMD:R_0805_2012Metric, F.Cu at (132.0, 130.0)
- added U500: LM393, Package_SO:SOIC-8_3.9x4.9mm_P1.27mm, F.Cu at (12.0, -20.0)
- added U600: MC33035, Package_SO:SOIC-24W_7.5x15.4mm_P1.27mm, F.Cu at (-1.00, -4.00)
- added U602: MC33039, Package_SO:SOIC-8_3.9x4.9mm_P1.27mm, F.Cu at (-6.00, 13.0)
- added U603: MOC8204, Package_DIP:DIP-6_W7.62mm_SMDSocket_SmallPads, F.Cu at (132.2, 123.5)
- added U604: MOC8204, Package_DIP:DIP-6_W7.62mm_SMDSocket_SmallPads, F.Cu at (109.2, 134.5)
- added U605: MOC8204, Package_DIP:DIP-6_W7.62mm_SMDSocket_SmallPads, F.Cu at (85.2, 123.5)
- C100, C101, C102: value 120x400V -> 120.0x400V
- D100: value 1N5626 -> KBU8M
- moved Q822 18.3 mm to (139.0, 141.0), turned to 210 degrees
- moved Q821 17.1 mm to (153.0, 130.0), turned to 225 degrees
Connections:
- net Net-(J1-Pad1) renamed /OKM
- D100 pad 2: Net-(C100-Pad2) -> Net-(D100-Pad2)
- D100 pad 3: (no net) -> Net-(D100-Pad3)
- D100 pad 4: (no net) -> Net-(C100-Pad2)
- J1 pad 2: Net-(J1-Pad2) -> /OKP
- J1 pad 4: Net-(D100-Pad1) -> Net-(D100-Pad2)

Commit message: plokstes paruosimas, nauji pdf-ai
Parts:
- added C201: 220x25V, Capacitor_THT:CP_Radial_D8.0mm_P2.50mm, F.Cu at (140.0, 52.0)
- added C300: 1.0x50V, Capacitor_THT:CP_Radial_D5.0mm_P2.50mm, F.Cu at (156.5, 50.2)
- added C609: 100x16V, Capacitor_THT:CP_Radial_D5.0mm_P2.50mm, F.Cu at (168.8, 103.7)
- added C802: 1.0x400V, Capacitor_THT:CP_Radial_D10.0mm_P5.00mm, F.Cu at (79.0, 101.0)
- added C803: 22x25V, Capacitor_THT:CP_Radial_D6.3mm_P2.50mm, F.Cu at (78.0, 125.0)
- added C804: 22x25V, Capacitor_THT:CP_Radial_D6.3mm_P2.50mm, F.Cu at (94.9, 139.0)
- added C805: 22x25V, Capacitor_THT:CP_Radial_D6.3mm_P2.50mm, F.Cu at (127.8, 139.0)
- added D106: LL4148, Diode_SMD:D_MiniMELF, F.Cu at (152.7, 53.0)
- added D600: 1N5818, Diode_SMD:D_SMA, F.Cu at (109.5, 135.1)
- added D601: 1N5818, Diode_SMD:D_SMA, F.Cu at (83.1, 127.3)
- added D602: 1N5818, Diode_SMD:D_SMA, F.Cu at (136.3, 127.9)
- added D805: MUR140, Diode_THT:D_DO-41_SOD81_P10.16mm_Horizontal, F.Cu at (78.0, 106.0)
- added D806: MUR140, Diode_THT:D_DO-41_SOD81_P10.16mm_Horizontal, F.Cu at (82.0, 116.0)
- added F1: Fuse, Fuse:Fuse_SunFuse-6HP, F.Cu at (99.0, 65.0)
- added P1: Conn_01x01, Connector_Pin:Pin_D1.0mm_L10.0mm, F.Cu at (80.0, 136.0)
- added P2: Conn_01x01, Connector_Pin:Pin_D1.0mm_L10.0mm, F.Cu at (114.0, 145.0)
- added P3: Conn_01x01, Connector_Pin:Pin_D1.0mm_L10.0mm, F.Cu at (145.0, 133.0)
- added R100.1: 100k, Resistor_SMD:R_1206_3216Metric, B.Cu at (53.0, 89.0)
- added R100.2: 100k, Resistor_SMD:R_1206_3216Metric, B.Cu at (58.0, 89.0)
- added R100.3: 100k, Resistor_SMD:R_1206_3216Metric, B.Cu at (63.0, 89.0)
- added R200: 180k, Resistor_THT:R_Axial_DIN0414_L11.9mm_D4.5mm_P15.24mm_Horizontal, F.Cu at (130.4, 44.6)
- added R202: 47R/5W, Resistor_THT:R_Axial_Power_L25.0mm_W9.0mm_P30.48mm, F.Cu at (100.0, 39.0)
- added R301: 490, Resistor_SMD:R_0805_2012Metric, F.Cu at (145.7, 50.8)
- added R604: 33k, Resistor_SMD:R_0805_2012Metric, F.Cu at (173.0, 87.5)
- added R702: 0.1/2W, Resistor_THT:R_Axial_DIN0411_L9.9mm_D3.6mm_P12.70mm_Horizontal, F.Cu at (74.0, 118.0)
- added TR1: SL12, Varistor:RV_Disc_D12mm_W3.9mm_P7.5mm, F.Cu at (58.0, 31.0)
- added U1: CNY17-1, Package_DIP:DIP-6_W7.62mm, F.Cu at (149.0, 39.8)
- added U606: NE555, Package_SO:SOIC-8_3.9x4.9mm_P1.27mm, F.Cu at (74.9, 88.9)
- added VP300: R_POT_TRIM, Potentiometer_THT:Potentiometer_ACP_CA6-H2,5_Horizontal, F.Cu at (137.0, 34.0)
- added Z200: 1N5245, Diode_THT:D_DO-35_SOD27_P7.62mm_Horizontal, F.Cu at (151.1, 55.6)
- added Z201: 1N5245, Diode_THT:D_DO-35_SOD27_P7.62mm_Horizontal, F.Cu at (148.3, 51.7)
- added Z203: 1N5245, Diode_THT:D_DO-35_SOD27_P7.62mm_Horizontal, F.Cu at (151.1, 58.3)
- added Z801: 1N4744, Diode_THT:D_DO-41_SOD81_P7.62mm_Horizontal, F.Cu at (89.5, 137.6)
- added Z804: 1N5352, Diode_THT:D_DO-41_SOD81_P10.16mm_Horizontal, F.Cu at (82.0, 91.0)
- added Z811: 1N4744, Diode_THT:D_DO-41_SOD81_P7.62mm_Horizontal, F.Cu at (121.7, 141.2)
- added Z821: 1N4744, Diode_THT:D_DO-41_SOD81_P7.62mm_Horizontal, F.Cu at (148.8, 124.6)
- D103, D104, D105, R206, R300, R805, R815, R825: moved to B.Cu
- H600, H601, H602: renamed from REF**; value PinHeader_1x03_P2.54mm_Vertical -> HALL
- J1: footprint jungtis:Jungtis -> valdiklio_footprints:Jungtis
- Q200: footprint Package_TO_SOT_THT:TO-220-3_Vertical -> Package_TO_SOT_THT:TO-220-3_Horizontal_TabDown
- Q201: value 2N4401 -> BC817; footprint Package_TO_SOT_THT:TO-92_Inline -> Package_TO_SOT_SMD:SOT-23
- Q202, Q300: value 2N3906 -> BC807; footprint Package_TO_SOT_THT:TO-92_Inline -> Package_TO_SOT_SMD:SOT-23
- moved U500 196.9 mm to (162.4, 107.1)
- moved U602 194.6 mm to (171.3, 93.3)
- moved U600 186.6 mm to (159.0, 92.0), turned to 180 degrees
- moved C605 149.0 mm to (173.1, 97.0), turned to 180 degrees
- moved C602 147.7 mm to (172.9, 89.6)
- moved C603 145.0 mm to (163.9, 103.5), turned to 180 degrees
- moved C600 140.8 mm to (167.9, 89.0), turned to 180 degrees
- moved C608 137.3 mm to (132.9, 116.7), turned to 45 degrees
- moved R605 137.0 mm to (169.7, 97.0)
- moved R501 136.5 mm to (156.2, 104.7), turned to 180 degrees
- moved C700 134.3 mm to (160.1, 86.9)
- moved R602 134.0 mm to (160.4, 103.5), turned to 180 degrees
- moved R502 133.5 mm to (156.2, 108.3)
- moved R500 132.0 mm to (156.2, 106.5)
- moved R607 130.3 mm to (136.0, 113.7), turned to 225 degrees
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Connections:
- H600 pad 1: (no net) -> /VCC
- H600 pad 2: (no net) -> Net-(H600-Pad2)
- H600 pad 3: (no net) -> GND
- H601 pad 1: (no net) -> /VCC
- H601 pad 2: (no net) -> Net-(H601-Pad2)
- H601 pad 3: (no net) -> GND
- H602 pad 1: (no net) -> /VCC
- H602 pad 2: (no net) -> Net-(H602-Pad2)
- H602 pad 3: (no net) -> GND
- J1 pad 1: /OKM -> Net-(F1-Pad2)
- J1 pad 2: /OKP -> Net-(D100-Pad2)
- J1 pad 3: /PE -> (no net)
- J1 pad 4: Net-(D100-Pad2) -> /OKP
- J1 pad 5: Net-(F1-Pad2) -> /OKM
- Q201 pad 1: Net-(C100-Pad2) -> Net-(C200-Pad2)
- Q201 pad 2: Net-(C200-Pad2) -> Net-(C100-Pad2)
- Q202 pad 1: Net-(C205-Pad1) -> Net-(C205-Pad2)
- Q202 pad 2: Net-(C205-Pad2) -> Net-(C205-Pad1)
- R302 pad 2: Net-(Q300-Pad2) -> Net-(Q300-Pad1)
- R303 pad 1: Net-(Q300-Pad1) -> Net-(Q300-Pad2)
- R303 pad 2: Net-(Q300-Pad2) -> Net-(Q300-Pad1)
- R304 pad 1: Net-(Q300-Pad2) -> Net-(Q300-Pad1)
- U602 pad 4: Net-(U602-Pad4) -> (no net)
- U603 pad 3: Net-(U603-Pad3) -> (no net)
- U604 pad 3: Net-(U604-Pad3) -> (no net)
- U605 pad 3: Net-(U605-Pad3) -> (no net)
Routing:
- added copper zone on F.Cu, net GND

Commit message: schemos ir plokstes paruosimas
Parts:
- added C610: 0.1, Capacitor_SMD:C_0805_2012Metric, F.Cu at (202.2, -37.9)
- added C611: 0.1, Capacitor_SMD:C_0805_2012Metric, F.Cu at (206.6, -37.9)
- added C612: 0.1, Capacitor_SMD:C_0805_2012Metric, F.Cu at (202.2, -34.9)
- added C613: 0.1, Capacitor_SMD:C_0805_2012Metric, F.Cu at (192.9, -22.4)
- added H600: SA, Connector_PinHeader_2.54mm:PinHeader_1x03_P2.54mm_Vertical, F.Cu at (193.0, -31.3)
- added H601: SB, Connector_PinHeader_2.54mm:PinHeader_1x03_P2.54mm_Vertical, F.Cu at (197.7, -31.3)
- added H602: SC, Connector_PinHeader_2.54mm:PinHeader_1x03_P2.54mm_Vertical, F.Cu at (213.9, -46.1)
- added J2: VB, TerminalBlock:TerminalBlock_bornier-2_P5.08mm, F.Cu at (203.2, -43.9)
- added J3: IF, Connector_PinHeader_2.54mm:PinHeader_1x10_P2.54mm_Vertical, F.Cu at (183.7, -46.1)
- added J4: IF, Connector_PinHeader_2.54mm:PinHeader_1x10_P2.54mm_Vertical, F.Cu at (188.4, -46.1)
- added J5: HALLS, Connector_PinHeader_2.54mm:PinHeader_1x05_P2.54mm_Vertical, F.Cu at (193.0, -46.1)
- added J6: HALLS, Connector_PinHeader_2.54mm:PinHeader_1x05_P2.54mm_Vertical, F.Cu at (197.7, -46.1)
Connections:
- net Net-(C700-Pad2) renamed /SENS
- J1 pad 3: (no net) -> /PE
- U1 pad 3: (no net) -> Net-(U1-Pad3)
- U1 pad 6: (no net) -> Net-(U1-Pad6)
- U600 pad 4: Net-(H600-Pad2) -> /~SA
- U600 pad 5: Net-(H601-Pad2) -> /~SB
- U600 pad 6: Net-(H602-Pad2) -> /~SC
- U602 pad 1: Net-(H600-Pad2) -> /~SA
- U602 pad 2: Net-(H602-Pad2) -> /~SC
- U602 pad 3: Net-(H601-Pad2) -> /~SB
- U602 pad 4: (no net) -> Net-(U602-Pad4)
- U603 pad 3: (no net) -> Net-(U603-Pad3)
- U604 pad 3: (no net) -> Net-(U604-Pad3)
- U605 pad 3: (no net) -> Net-(U605-Pad3)
- U606 pad 5: (no net) -> Net-(U606-Pad5)
- U606 pad 7: (no net) -> Net-(U606-Pad7)

Commit message: 2019.10.10
Parts:
- removed C200, C205: 1nF, Capacitor_SMD:C_0805_2012Metric
- removed C201: 220x25V, Capacitor_THT:CP_Radial_D8.0mm_P2.50mm
- removed C300: 1.0x50V, Capacitor_THT:CP_Radial_D5.0mm_P2.50mm
- removed C600, C602, C603, C610, C611, C612, C613: 0.1, Capacitor_SMD:C_0805_2012Metric
- removed C601, C801: 10n, Capacitor_SMD:C_0805_2012Metric
- removed C604: 47n, Capacitor_SMD:C_0805_2012Metric
- removed C605: 22n, Capacitor_SMD:C_0805_2012Metric
- removed C606, C607, C608: 2n2, Capacitor_SMD:C_0805_2012Metric
- removed C609: 100x16V, Capacitor_THT:CP_Radial_D5.0mm_P2.50mm
- removed C700: 4n7, Capacitor_SMD:C_0805_2012Metric
- removed C802: 1.0x400V, Capacitor_THT:CP_Radial_D10.0mm_P5.00mm
- removed C803, C804, C805: 22x25V, Capacitor_THT:CP_Radial_D6.3mm_P2.50mm
- removed D100: KBU8M, Diode_THT:Diode_Bridge_Vishay_KBU
- removed D103, D105, D300: LL4005, Diode_SMD:D_MELF
- removed D104: LL4006, Diode_SMD:D_MELF
- removed D106, D801, D811, D821: LL4148, Diode_SMD:D_MiniMELF
- removed D600, D601, D602: 1N5818, Diode_SMD:D_SMA
- removed D805, D806: MUR140, Diode_THT:D_DO-41_SOD81_P10.16mm_Horizontal
- removed the H600 at (193.0, -31.3)
- removed the H601 at (197.7, -31.3)
- removed the H602 at (213.9, -46.1)
- removed Q200: IRF830, Package_TO_SOT_THT:TO-220-3_Horizontal_TabDown
- removed Q201: BC817, Package_TO_SOT_SMD:SOT-23
- removed Q202, Q300: BC807, Package_TO_SOT_SMD:SOT-23
- removed Q821, Q822: IRF830, valdiklio_footprints:TO-220-3_Vertical
- removed R100.1, R100.2, R100.3: 100k, Resistor_SMD:R_1206_3216Metric
- removed R200: 180k, Resistor_THT:R_Axial_DIN0414_L11.9mm_D4.5mm_P15.24mm_Horizontal
- removed R201, R204, R304, R602: 10k, Resistor_SMD:R_0805_2012Metric
- removed R202: 47R/5W, Resistor_THT:R_Axial_Power_L25.0mm_W9.0mm_P30.48mm
- removed R206, R305: 2.2k, Resistor_SMD:R_0805_2012Metric
- removed R207, R300, R700, R701: 1k, Resistor_SMD:R_0805_2012Metric
- removed R301: 490, Resistor_SMD:R_0805_2012Metric
- removed R302, R500, R502: 20k, Resistor_SMD:R_0805_2012Metric
- removed R303, R801, R811, R821: 1M, Resistor_SMD:R_0805_2012Metric
- removed R306, R604: 33k, Resistor_SMD:R_0805_2012Metric
- removed R307: 22k, Resistor_SMD:R_0805_2012Metric
- removed R501: 4.5k, Resistor_SMD:R_0805_2012Metric
- removed R600: 4.7k, Resistor_SMD:R_0805_2012Metric
- removed R601: 150k, Resistor_SMD:R_0805_2012Metric
- removed R603, R607, R608: 1.8k, Resistor_SMD:R_0805_2012Metric
- removed R605: 7.5k, Resistor_SMD:R_0805_2012Metric
- removed R606: 49k, Resistor_SMD:R_0805_2012Metric
- removed R702: 0.1/2W, Resistor_THT:R_Axial_DIN0411_L9.9mm_D3.6mm_P12.70mm_Horizontal
- removed R803, R813, R823: 72R, Resistor_SMD:R_0805_2012Metric
- removed R804, R814, R824: 100R, Resistor_SMD:R_0805_2012Metric
- removed R805, R808, R815, R825: 18k, Resistor_SMD:R_0805_2012Metric
- removed the REF** at (127.0, 107.0)
- removed the REF** at (87.0, 96.0)
- removed TR1: SL12, Varistor:RV_Disc_D12mm_W3.9mm_P7.5mm
- removed U500: LM393, Package_SO:SOIC-8_3.9x4.9mm_P1.27mm
- removed U600: MC33035, Package_SO:SOIC-24W_7.5x15.4mm_P1.27mm
- removed U602: MC33039, Package_SO:SOIC-8_3.9x4.9mm_P1.27mm
- removed U603, U604, U605: MOC8204, Package_DIP:DIP-6_W7.62mm_SMDSocket_SmallPads
- removed U606: NE555, Package_SO:SOIC-8_3.9x4.9mm_P1.27mm
- removed VP300: R_POT_TRIM, Potentiometer_THT:Potentiometer_ACP_CA6-H2,5_Horizontal
- removed Z200, Z201, Z203: 1N5245, Diode_THT:D_DO-35_SOD27_P7.62mm_Horizontal
- removed Z801, Z811, Z821: 1N4744, Diode_THT:D_DO-41_SOD81_P7.62mm_Horizontal
- removed Z804: 1N5352, Diode_THT:D_DO-41_SOD81_P10.16mm_Horizontal
- added C1: 22n, Capacitor_SMD:C_0805_2012Metric, F.Cu at (17.7, -41.6)
- added C10: 100x16V, Capacitor_THT:CP_Radial_D5.0mm_P2.50mm, F.Cu at (-4.90, -22.0)
- added C11: 100n, Capacitor_SMD:C_0805_2012Metric, F.Cu at (17.7, -47.5)
- added C12: 100x16V, Capacitor_THT:CP_Radial_D6.3mm_P2.50mm, F.Cu at (-23.3, -7.72)
- added C13: 0.1, Capacitor_SMD:C_0805_2012Metric, F.Cu at (17.7, -44.5)
- added C14: 0.1, Capacitor_SMD:C_0805_2012Metric, F.Cu at (-34.9, 10.1)
- added C15: 100n, Capacitor_SMD:C_0805_2012Metric, F.Cu at (-24.8, 1.93)
- added C16: 0.1, Capacitor_SMD:C_0805_2012Metric, F.Cu at (19.1, -29.2)
- added C17: 0.1, Capacitor_SMD:C_0805_2012Metric, F.Cu at (-17.0, 0.18)
- added C18: 100n, Capacitor_SMD:C_0805_2012Metric, F.Cu at (-24.8, 4.88)
- added C19: 100n, Capacitor_SMD:C_0805_2012Metric, F.Cu at (-8.15, 0.18)
- added C2: 120x400V, Capacitor_THT:CP_Radial_D22.0mm_P10.00mm_SnapIn, F.Cu at (-91.4, -41.7)
- added C20: 100x16V, Capacitor_THT:CP_Radial_D6.3mm_P2.50mm, F.Cu at (9.85, -37.6)
- added C21: 2n2, Capacitor_SMD:C_0805_2012Metric, F.Cu at (14.6, -26.3)
- added C22: 2n2, Capacitor_SMD:C_0805_2012Metric, F.Cu at (5.93, -18.2)
- added C23: 2n2, Capacitor_SMD:C_0805_2012Metric, F.Cu at (-26.1, 13.7)
- added C24: 4n7, Capacitor_SMD:C_0805_2012Metric, F.Cu at (-7.91, -3.47)
- added C25: 10n, Capacitor_SMD:C_0805_2012Metric, F.Cu at (-21.7, 9.03)
- added C26: 1.0x400V, Capacitor_THT:CP_Radial_D10.0mm_P5.00mm, F.Cu at (-61.8, 4.23)
- added C27: 0.1, Capacitor_SMD:C_0805_2012Metric, F.Cu at (-3.50, -8.37)
- added C28: 0.1, Capacitor_SMD:C_0805_2012Metric, F.Cu at (10.6, -21.2)
- added C29: 22x25V, Capacitor_THT:CP_Radial_D6.3mm_P2.50mm, F.Cu at (-42.3, 11.7)
- added C3: 4.7x400V, Capacitor_THT:CP_Radial_D10.0mm_P5.00mm, F.Cu at (-57.2, -8.02)
- added C30: 0.1, Capacitor_SMD:C_0805_2012Metric, F.Cu at (1.52, -11.3)
- added C31: 22x25V, Capacitor_THT:CP_Radial_D6.3mm_P2.50mm, F.Cu at (-15.3, -5.22)
- added C32: 22x25V, Capacitor_THT:CP_Radial_D6.3mm_P2.50mm, F.Cu at (-3.49, -29.2)
- added C4: 120x400V, Capacitor_THT:CP_Radial_D22.0mm_P10.00mm_SnapIn, F.Cu at (-67.2, -41.7)
- added C5: 4.7x400V, Capacitor_THT:CP_Radial_D10.0mm_P5.00mm, F.Cu at (-22.6, -32.9)
- added C6: 120x400V, Capacitor_THT:CP_Radial_D22.0mm_P10.00mm_SnapIn, F.Cu at (-42.9, -41.7)
- added C7: 47n, Capacitor_SMD:C_0805_2012Metric, F.Cu at (-80.7, 14.0)
- added C8: 10n, Capacitor_SMD:C_0805_2012Metric, F.Cu at (-19.3, -40.3)
- added C9: 1.0x50V, Capacitor_THT:CP_Radial_D5.0mm_P2.50mm, F.Cu at (-9.62, -14.1)
- added D1: D, Diode_THT:D_DO-201AD_P15.24mm_Horizontal, F.Cu at (-101.1, 4.88)
- added D10: 1N5818, Diode_SMD:D_SMA, F.Cu at (17.0, -51.2)
- added D11: 1N5818, Diode_SMD:D_SMA, F.Cu at (-73.9, 14.3)
- added D12: 1N5818, Diode_SMD:D_SMA, F.Cu at (-10.3, -29.8)
- added D13: LL4148, Diode_SMD:D_MiniMELF, F.Cu at (-30.2, 2.08)
- added D14: LL4148, Diode_SMD:D_MiniMELF, F.Cu at (4.86, -27.2)
- added D15: LL4148, Diode_SMD:D_MiniMELF, F.Cu at (-22.4, -2.17)
- added D16: MUR140, Diode_THT:D_DO-41_SOD81_P10.16mm_Horizontal, F.Cu at (-57.0, -22.7)
- added D17: MUR140, Diode_THT:D_DO-41_SOD81_P10.16mm_Horizontal, F.Cu at (-84.1, -1.12)
- added D2: D, Diode_THT:D_DO-201AD_P15.24mm_Horizontal, F.Cu at (-96.5, -19.8)
- added D3: D, Diode_THT:D_DO-201AD_P15.24mm_Horizontal, F.Cu at (-76.5, -26.6)
- added D4: D, Diode_THT:D_DO-201AD_P15.24mm_Horizontal, F.Cu at (-96.5, -26.6)
- added D5: LL4005, Diode_SMD:D_MELF, F.Cu at (-33.2, 6.53)
- added D6: LL4005, Diode_SMD:D_MELF, F.Cu at (5.61, -31.0)
- added D7: LL4005, Diode_SMD:D_MELF, F.Cu at (-29.5, -1.67)
- added D8: UF4005, Diode_THT:D_DO-41_SOD81_P10.16mm_Horizontal, F.Cu at (-65.0, -15.9)
- added D9: 12V, Diode_SMD:D_MiniMELF, F.Cu at (-86.1, 14.1)
- added F2: 3A, Fuse:Fuseholder_TR5_Littelfuse_No560_No460, F.Cu at (-34.1, -10.8)
- added H1: SA, Connector_PinHeader_2.54mm:PinHeader_1x03_P2.54mm_Vertical, F.Cu at (-12.0, -39.5)
- added H2: SB, Connector_PinHeader_2.54mm:PinHeader_1x03_P2.54mm_Vertical, F.Cu at (4.72, -45.6)
- added H3: SC, Connector_PinHeader_2.54mm:PinHeader_1x03_P2.54mm_Vertical, F.Cu at (-35.7, -2.97)
- added J1: HALLS, Connector_PinHeader_2.54mm:PinHeader_1x05_P2.54mm_Vertical, F.Cu at (-67.7, -8.97)
- added L1: 1mH, Inductor_SMD:L_Vishay_IHSM-3825, F.Cu at (-78.0, -7.27)
- added L2: 1mH/280mA, Inductor_THT:L_Radial_D7.8mm_P5.00mm_Fastron_07HCP, F.Cu at (-14.4, -22.3)
- added Q1: BC807, Package_TO_SOT_SMD:SOT-23, F.Cu at (3.92, -36.0)
- added Q2: IRF830, valdiklio_footprints:TO-220-3_Vertical, F.Cu at (607.0, 132.0)
- added Q3: IRF830, valdiklio_footprints:TO-220-3_Vertical, F.Cu at (593.0, 143.0)
- added R1: 1k, Resistor_SMD:R_0805_2012Metric, F.Cu at (15.1, -23.3)
- added R10: 2.2k, Resistor_SMD:R_0805_2012Metric, F.Cu at (3.89, -24.1)
- added R11: 49k, Resistor_SMD:R_0805_2012Metric, F.Cu at (-2.89, -17.2)
- added R12: 150k, Resistor_SMD:R_0805_2012Metric, F.Cu at (11.7, -32.2)
- added R13: 33k, Resistor_SMD:R_0805_2012Metric, F.Cu at (-16.0, 6.08)
- added R14: 22k, Resistor_SMD:R_0805_2012Metric, F.Cu at (16.1, -32.2)
- added R15: 4.7k, Resistor_SMD:R_0805_2012Metric, F.Cu at (1.52, -17.2)
- added R16: 20k, Resistor_SMD:R_0805_2012Metric, F.Cu at (-2.89, -14.3)
- added R17: 4.5k, Resistor_SMD:R_0805_2012Metric, F.Cu at (-30.5, 10.1)
- added R18: 20k, Resistor_SMD:R_0805_2012Metric, F.Cu at (1.83, -21.2)
- added R19: 10k, Resistor_SMD:R_0805_2012Metric, F.Cu at (-26.1, 7.83)
- added R2: 7.5k, Resistor_SMD:R_0805_2012Metric, F.Cu at (8.30, -24.1)
- added R20: 4k7, Resistor_SMD:R_0805_2012Metric, F.Cu at (-20.4, 3.13)
- added R21: 10k, Resistor_SMD:R_0805_2012Metric, F.Cu at (-26.1, 10.8)
- added R22: 1.8k, Resistor_SMD:R_0805_2012Metric, F.Cu at (6.24, -21.2)
- added R23: 1.8k, Resistor_SMD:R_0805_2012Metric, F.Cu at (-2.89, -11.3)
- added R24: 1.8k, Resistor_SMD:R_0805_2012Metric, F.Cu at (-20.4, 6.08)
- added R25: 1k, Resistor_SMD:R_0805_2012Metric, F.Cu at (-7.91, -6.42)
- added R26: 18k, Resistor_SMD:R_0805_2012Metric, F.Cu at (-12.6, 0.18)
- added R27: 100R, Resistor_SMD:R_0805_2012Metric, F.Cu at (-16.0, 3.13)
- added R28: 100R, Resistor_SMD:R_0805_2012Metric, F.Cu at (1.52, -14.3)
- added R29: 100R, Resistor_SMD:R_0805_2012Metric, F.Cu at (-7.91, -9.37)
- added R3: 8R2/2W, Resistor_THT:R_Axial_DIN0411_L9.9mm_D3.6mm_P12.70mm_Horizontal, F.Cu at (-76.9, -20.6)
- added R30: 1k, Resistor_SMD:R_0805_2012Metric, F.Cu at (-51.3, -0.77)
- added R31: 1M, Resistor_SMD:R_0805_2012Metric, F.Cu at (-21.7, 12.0)
- added R32: 72R, Resistor_SMD:R_0805_2012Metric, F.Cu at (14.6, -29.2)
- added R33: 1M, Resistor_SMD:R_0805_2012Metric, F.Cu at (-3.50, -5.42)
- added R34: 72R, Resistor_SMD:R_0805_2012Metric, F.Cu at (-17.3, 9.03)
- added R35: 1M, Resistor_SMD:R_0805_2012Metric, F.Cu at (5.93, -15.3)
- added R36: 72R, Resistor_SMD:R_0805_2012Metric, F.Cu at (-11.6, 3.13)
- added R37: 18k, Resistor_SMD:R_0805_2012Metric, F.Cu at (19.1, -26.3)
- added R38: 18k, Resistor_SMD:R_0805_2012Metric, F.Cu at (10.3, -18.2)
- added R39: 18k, Resistor_SMD:R_0805_2012Metric, F.Cu at (0.91, -8.37)
- added R4: 490, Resistor_SMD:R_0805_2012Metric, F.Cu at (-34.9, 13.1)
- added R40: 0.1/2W, Resistor_THT:R_Axial_DIN0411_L9.9mm_D3.6mm_P12.70mm_Horizontal, F.Cu at (-56.9, -27.4)
- added R5: 33k, Resistor_SMD:R_0805_2012Metric, F.Cu at (17.2, -38.6)
- added R6: 20k, Resistor_SMD:R_0805_2012Metric, F.Cu at (10.2, -27.4)
- added R7: 10k, Resistor_SMD:R_0805_2012Metric, F.Cu at (17.2, -35.7)
- added R8: 220k, Resistor_THT:R_Axial_DIN0411_L9.9mm_D3.6mm_P12.70mm_Horizontal, F.Cu at (-81.5, -13.9)
- added R9: 1M, Resistor_SMD:R_0805_2012Metric, F.Cu at (-30.5, 13.1)
- added REF**: MountingHole_2.7mm, MountingHole:MountingHole_2.7mm, F.Cu at (581.0, 109.0)
- added REF**: MountingHole_2.7mm, MountingHole:MountingHole_2.7mm, F.Cu at (541.0, 98.0)
- added RV1: Varistor, Varistor:RV_Disc_D9mm_W4mm_P5mm, F.Cu at (-50.8, 4.03)
- added RV2: Varistor, Varistor:RV_Disc_D9mm_W4mm_P5mm, F.Cu at (5.17, -51.7)
- added TH1: 33R, Varistor:RV_Disc_D9mm_W4mm_P5mm, F.Cu at (-63.8, 11.8)
- added U10: MOC8204, Package_DIP:DIP-6_W7.62mm_SMDSocket_SmallPads, F.Cu at (-36.3, -21.0)
- added U11: MOC8204, Package_DIP:DIP-6_W7.62mm_SMDSocket_SmallPads, F.Cu at (-3.48, -48.8)
- added U2: MC33039, Package_SO:SOIC-8_3.9x4.9mm_P1.27mm, F.Cu at (11.3, -44.7)
- added U3: LNK304G, Package_DIP:PowerIntegrations_SMD-8B, F.Cu at (-15.4, -47.6)
- added U4: PC817, Package_DIP:DIP-4_W10.16mm_LongPads, F.Cu at (-101.5, 10.3)
- added U5: MC33035, Package_SO:SOIC-24W_7.5x15.4mm_P1.27mm, F.Cu at (-92.4, -7.97)
- added U6: LM393, Package_SO:SOIC-8_3.9x4.9mm_P1.27mm, F.Cu at (-21.9, -14.9)
- added U7: SIP21106, Package_TO_SOT_SMD:SOT-23-5, F.Cu at (-40.6, 4.53)
- added U8: NE555, Package_SO:SOIC-8_3.9x4.9mm_P1.27mm, F.Cu at (-49.3, 11.0)
- added U9: MOC8204, Package_DIP:DIP-6_W7.62mm_SMDSocket_SmallPads, F.Cu at (-43.0, -11.7)
- added VP1: R_POT_TRIM, Potentiometer_THT:Potentiometer_ACP_CA6-H2,5_Horizontal, F.Cu at (-16.0, -15.8)
- added Z1: 1N5352, Diode_THT:D_DO-41_SOD81_P10.16mm_Horizontal, F.Cu at (-40.3, -27.8)
- added Z2: 1N4744, Diode_THT:D_DO-41_SOD81_P7.62mm_Horizontal, F.Cu at (-76.1, 9.88)
- added Z3: 1N4744, Diode_THT:D_DO-41_SOD81_P7.62mm_Horizontal, F.Cu at (-76.1, 5.63)
- added Z4: 1N4744, Diode_THT:D_DO-41_SOD81_P7.62mm_Horizontal, F.Cu at (-87.4, 10.4)
- F1: value Fuse -> 5A; footprint Fuse:Fuse_SunFuse-6HP -> Fuse:Fuseholder_TR5_Littelfuse_No560_No460
- J2: value VB -> IF; footprint TerminalBlock:TerminalBlock_bornier-2_P5.08mm -> Connector_PinHeader_2.54mm:PinHeader_1x10_P2.54mm_Vertical
- J3: value IF -> HALLS; footprint Connector_PinHeader_2.54mm:PinHeader_1x10_P2.54mm_Vertical -> Connector_PinHeader_2.54mm:PinHeader_1x05_P2.54mm_Vertical
- J5: value HALLS -> GND; footprint Connector_PinHeader_2.54mm:PinHeader_1x05_P2.54mm_Vertical -> Connector_PinHeader_2.54mm:PinHeader_1x04_P2.54mm_Vertical
- J6: value HALLS -> VB; footprint Connector_PinHeader_2.54mm:PinHeader_1x05_P2.54mm_Vertical -> TerminalBlock:TerminalBlock_bornier-2_P5.08mm
- moved H600 454.0 mm to (593.7, 72.4)
- moved Q6 454.0 mm to (538.7, 145.2)
- moved ? 454.0 mm to (514.0, 126.0)
- moved ? 454.0 mm to (614.0, 126.0)
- moved C100 454.0 mm to (507.0, 103.0)
- moved C101 454.0 mm to (507.0, 79.0)
- moved C102 454.0 mm to (517.0, 58.0)
- moved H601 454.0 mm to (599.5, 89.5)
- moved H602 454.0 mm to (596.2, 107.3)
- moved J1 454.0 mm to (564.0, 32.0)
- moved Q5 454.0 mm to (556.9, 150.5)
- moved Q7 454.0 mm to (524.0, 135.0)
- moved REF** 454.0 mm to (598.0, 101.0)
- moved REF** 454.0 mm to (598.0, 83.0)
- moved REF** 454.0 mm to (571.0, 69.0)
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- renumbered Q811 to Q4, Q812 to Q5, Q801 to Q6, Q802 to Q7
Connections:
- F1 pad 2: Net-(F1-Pad2) -> /ACL
- J2 pad 1: /+U -> /AB
- J2 pad 2: GND -> /AT
- J3 pad 1: /AB -> /VCC
- J3 pad 2: /AT -> /~SA
- J3 pad 3: /BB -> /~SB
- J3 pad 4: /BT -> /~SC
- J3 pad 5: /CB -> GND
- J4 pad 1: /AB -> /VCC
- J4 pad 2: /AT -> /VCC
- J4 pad 3: /BB -> /AB
- J4 pad 4: /BT -> /AT
- J4 pad 5: /CB -> /BB
- J4 pad 6: /CT -> /BT
- J4 pad 7: Net-(J4-Pad7) -> /CB
- J4 pad 8: Net-(J4-Pad8) -> /CT
- J5 pad 1: /VCC -> GND
- J5 pad 2: /~SA -> GND
- J5 pad 3: /~SB -> GND
- J5 pad 4: /~SC -> (no net)
- J6 pad 1: /VCC -> /+U
- J6 pad 2: /~SA -> GND
- Q4 pad 2: /+U -> Net-(Q4-Pad2)
- Q4 pad 3: Net-(P2-Pad1) -> Net-(P1-Pad1)
- Q5 pad 2: Net-(P2-Pad1) -> Net-(P1-Pad1)
- Q6 pad 2: /+U -> Net-(Q6-Pad2)
- Q6 pad 3: Net-(P1-Pad1) -> Net-(P3-Pad1)
- Q7 pad 2: Net-(P1-Pad1) -> Net-(P3-Pad1)
