File: variklio_valdiklis_mc33035.sch (KiCad schematic (older format))
At the start: 129 parts, among them J1 Conn_01x05, J2 VB, J3 IF, J4 IF, J5 HALLS, J6 HALLS, P1 Conn_01x01, P2 Conn_01x01, P3 Conn_01x01, Q200 IRF830, Q201 BC817, Q202 BC807, Q300 BC807, Q801 IRF830, Q802 IRF830, Q811 IRF830, Q812 IRF830, Q821 IRF830, Q822 IRF830, U1 CNY17-1, U500 LM393, U600 MC33035, U602 MC33039, U603 MOC8204, U604 MOC8204, U605 MOC8204, U606 NE555

Commit message: schema stm32f103c8t
Parts:
- added R826, R827, R828: R, symbol resistors_us:R_0R22_2W_5%
- H600, H601, H602: symbol variklio_valdiklis-rescue:A1101ELHL-Sensor_Magnetic -> variklio_valdiklis_mc33035-rescue:A1101ELHL-Sensor_Magnetic-variklio_valdiklis-rescue
- U600: symbol variklio_valdiklis-rescue:MC33035-ics -> variklio_valdiklis_mc33035-rescue:MC33035-ics-variklio_valdiklis-rescue
- U602: symbol variklio_valdiklis-rescue:MC33039-ics -> variklio_valdiklis_mc33035-rescue:MC33039-ics-variklio_valdiklis-rescue
- gave numbers to parts that had none: 2
Connections:
- wire segments 475 -> 478
Other:
- moved on the sheet: C606, C700, C801, C802, C803, C804, C805, D600, D601, D801, D805, D806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

Commit message: stm32f103c8tx schemos ir plokstes ruosimas
Parts:
- R826, R827, R828: symbol resistors_us:R_0R22_2W_5% -> variklio_valdiklis_mc33035-rescue:R_0R22_2W_5%-resistors_us
Changed lines of the file:
@@
 EESchema Schematic File Version 4
 LIBS:variklio_valdiklis_mc33035-cache
-EELAYER 29 0
+EELAYER 30 0
 EELAYER END
 $Descr A3 16535 11693
@@
 	5200 10500 5200 10000
 $Comp
-L resistors_us:R_0R22_2W_5% R826
+L variklio_valdiklis_mc33035-rescue:R_0R22_2W_5%-resistors_us R826
 U 1 1 5DA65689
 P 14500 2900
@@
 	14650 2900 14950 2900
 $Comp
-L resistors_us:R_0R22_2W_5% R827
+L variklio_valdiklis_mc33035-rescue:R_0R22_2W_5%-resistors_us R827
 U 1 1 5DA69207
 P 14500 4500
@@
 	14350 4500 14050 4500
 $Comp
-L resistors_us:R_0R22_2W_5% R828
+L variklio_valdiklis_mc33035-rescue:R_0R22_2W_5%-resistors_us R828
 U 1 1 5DA69BB3
 P 14500 6100

Commit message: 2019.10.10
Parts:
- removed C100, C101, C102: 120.0x400V, Capacitor_THT:CP_Radial_D22.0mm_P10.00mm_SnapIn, symbol Device:CP
- removed C200, C205: 1nF, Capacitor_SMD:C_0805_2012Metric, symbol Device:C
- removed C201: 220x25V, Capacitor_THT:CP_Radial_D8.0mm_P2.50mm, symbol Device:CP
- removed C611, C612: 0.1, Capacitor_SMD:C_0805_2012Metric, symbol Device:C
- removed D100: KBU8M, Diode_THT:Diode_Bridge_Vishay_KBU, symbol Diode_Bridge:KBU8M
- removed D103, D105, D300: LL4005, Diode_SMD:D_MELF, symbol Device:D
- removed D104: LL4006, Diode_SMD:D_MELF, symbol Device:D
- removed D106: LL4148, Diode_SMD:D_MiniMELF, symbol Device:D
- removed J1: Conn_01x05, valdiklio_footprints:Jungtis, symbol Connector_Generic:Conn_01x05
- removed J2, J8: VB, TerminalBlock:TerminalBlock_bornier-2_P5.08mm, symbol Connector_Generic:Conn_01x02
- removed Q200: IRF830, Package_TO_SOT_THT:TO-220-3_Horizontal_TabDown, symbol Transistor_FET:IRF740
- removed Q201: BC817, Package_TO_SOT_SMD:SOT-23, symbol Transistor_BJT:BC817
- removed Q202, Q300: BC807, Package_TO_SOT_SMD:SOT-23, symbol Transistor_BJT:BC807
- removed R100.1, R100.2, R100.3: 100k, Resistor_SMD:R_1206_3216Metric, symbol Device:R_US
- removed R200: 180k, Resistor_THT:R_Axial_DIN0414_L11.9mm_D4.5mm_P15.24mm_Horizontal, symbol Device:R
- removed R201, R204: 10k, Resistor_SMD:R_0805_2012Metric, symbol Device:R
- removed R202: 47R/5W, Resistor_THT:R_Axial_Power_L25.0mm_W9.0mm_P30.48mm, symbol Device:R_US
- removed R206, R305: 2.2k, Resistor_SMD:R_0805_2012Metric, symbol Device:R
- removed R207, R300: 1k, Resistor_SMD:R_0805_2012Metric, symbol Device:R
- removed R302: 20k, Resistor_SMD:R_0805_2012Metric, symbol Device:R
- removed R307: 22k, Resistor_SMD:R_0805_2012Metric, symbol Device:R
- removed TR1: SL12, Varistor:RV_Disc_D12mm_W3.9mm_P7.5mm, symbol Device:R_US
- removed Z200, Z201, Z203: 1N5245, Diode_THT:D_DO-35_SOD27_P7.62mm_Horizontal, symbol Device:D_Zener
- added C11, C15, C18, C19: 100n, Capacitor_SMD:C_0805_2012Metric, symbol variklio_valdiklis_stm32F103-rescue:C-Device
- added C12, C20: 100x16V, Capacitor_THT:CP_Radial_D6.3mm_P2.50mm, symbol variklio_valdiklis_stm32F103-rescue:CP-Device
- added C2, C4, C6: 120x400V, Capacitor_THT:CP_Radial_D22.0mm_P10.00mm_SnapIn, symbol variklio_valdiklis_stm32F103-rescue:CP-Device
- added C27, C28: 0.1, Capacitor_SMD:C_0805_2012Metric, symbol Device:C
- added C3, C5: 4.7x400V, Capacitor_THT:CP_Radial_D10.0mm_P5.00mm, symbol variklio_valdiklis_stm32F103-rescue:CP-Device
- added D1, D2, D3, D4: D, Diode_THT:D_DO-201AD_P15.24mm_Horizontal, symbol variklio_valdiklis_stm32F103-rescue:D-Device
- added D5: LL4005, Diode_SMD:D_MELF, symbol Device:D
- added D6, D7: LL4005, Diode_SMD:D_MELF, symbol variklio_valdiklis_stm32F103-rescue:D-Device
- added D8: UF4005, Diode_THT:D_DO-41_SOD81_P10.16mm_Horizontal, symbol variklio_valdiklis_stm32F103-rescue:D-Device
- added D9: 12V, Diode_SMD:D_MiniMELF, symbol variklio_valdiklis_stm32F103-rescue:D_Zener-Device
- added F2: 3A, Fuse:Fuseholder_TR5_Littelfuse_No560_No460, symbol Device:Fuse
- added L1: 1mH, Inductor_SMD:L_Vishay_IHSM-3825, symbol variklio_valdiklis_stm32F103-rescue:L-Device
- added L2: 1mH/280mA, Inductor_THT:L_Radial_D7.8mm_P5.00mm_Fastron_07HCP, symbol Device:L_Core_Iron
- added Q1: BC807, Package_TO_SOT_SMD:SOT-23, symbol Transistor_BJT:BC807
- added R1: 1k, Resistor_SMD:R_0805_2012Metric, symbol Device:R
- added R10: 2.2k, Resistor_SMD:R_0805_2012Metric, symbol Device:R
- added R14: 22k, Resistor_SMD:R_0805_2012Metric, symbol Device:R
- added R20: 4k7, Resistor_SMD:R_0805_2012Metric, symbol variklio_valdiklis_stm32F103-rescue:R-Device
- added R21: 10k, Resistor_SMD:R_0805_2012Metric, symbol variklio_valdiklis_stm32F103-rescue:R-Device
- added R3: 8R2/2W, Resistor_THT:R_Axial_DIN0411_L9.9mm_D3.6mm_P12.70mm_Horizontal, symbol variklio_valdiklis_stm32F103-rescue:R-Device
- added R6: 20k, Resistor_SMD:R_0805_2012Metric, symbol Device:R
- added R8: 220k, Resistor_THT:R_Axial_DIN0411_L9.9mm_D3.6mm_P12.70mm_Horizontal, symbol variklio_valdiklis_stm32F103-rescue:R-Device
- added RV1, RV2: Varistor, Varistor:RV_Disc_D9mm_W4mm_P5mm, symbol Device:Varistor
- added TH1: 33R, Varistor:RV_Disc_D9mm_W4mm_P5mm, symbol Device:Thermistor_PTC
- added U3: LNK304G, Package_DIP:PowerIntegrations_SMD-8B, symbol variklio_valdiklis_stm32F103-rescue:LNK304G-Regulator_Switching
- added U4: PC817, Package_DIP:DIP-4_W10.16mm_LongPads, symbol variklio_valdiklis_stm32F103-rescue:PC817-Isolator
- added U7: SIP21106, Package_TO_SOT_SMD:SOT-23-5, symbol variklio_valdiklis_stm32F103-rescue:USTAB_SIP21106-DT-33-disc
- F1: value Fuse -> 5A; footprint Fuse:Fuse_SunFuse-6HP -> Fuse:Fuseholder_TR5_Littelfuse_No560_No460
- renumbered C605 to C1, C609 to C10, C600 to C13, C602 to C14, C603 to C16, C610 to C17, C607 to C21, C606 to C22, C608 to C23, C700 to C24, C801 to C25, C802 to C26, C803 to C29, C613 to C30, C804 to C31, C805 to C32, C604 to C7, C601 to C8, C300 to C9, D602 to D10, D600 to D11, D601 to D12, D821 to D13, D811 to D14, D801 to D15, D805 to D16, D806 to D17, H600 to H1, H601 to H2, H602 to H3, J5 to J1, J3 to J2, J6 to J3, J7 to J5, P2 to P1, P3 to P2, P1 to P3, Q821 to Q2, Q822 to Q3, Q811 to Q4, Q812 to Q5, Q801 to Q6, Q802 to Q7, R606 to R11, R601 to R12, R306 to R13, R600 to R15, R500 to R16, R501 to R17, R502 to R18, R602 to R19, R605 to R2, R608 to R22, R603 to R23, R607 to R24, R700 to R25, R808 to R26, R824 to R27, R814 to R28, R804 to R29, R701 to R30, R821 to R31, R823 to R32, R811 to R33, R813 to R34, R801 to R35, R803 to R36, R825 to R37, R815 to R38, R805 to R39, R301 to R4, R702 to R40, R826 to R41, R827 to R42, R828 to R43, R604 to R5, R304 to R7, R303 to R9, TR2 to TR1, U604 to U10, U605 to U11, U602 to U2, U600 to U5, U500 to U6, U606 to U8, U603 to U9, VP300 to VP1, Z804 to Z1, Z821 to Z2, Z811 to Z3, Z801 to Z4
Connections:
- net labels added: 3VDC, ACL, ACN, VB
- net labels removed: +V, PE
- wire segments 478 -> 494
Other:
- moved on the sheet: C1, C10, C13, C14, C16, C17, C21, C22, C23, C24, C25, C26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
