File: variklio_valdiklis_stm32F103.kicad_pcb (KiCad board)
At the start: 2 copper layers, 134 x 134 mm, 67 parts, among them J1 Conn_01x05, J3 HALLS, P1 Conn_01x01, Q4 IRF830, Q5 IRF830, Q6 IRF830, Q7 IRF830, Q8 IRF830, Q801 IRF830, Q802 IRF830, Q811 IRF830, Q812 IRF830, Q821 IRF830, Q822 IRF830, Q9 IRF830, U1 STM32F103C8Tx, U5 LNK304G, U6 PC817

Commit message: stm32f103c8tx schemos ir plokstes ruosimas
Parts:
- removed the H1 at (44.3, -24.2)
- removed the H2 at (24.1, -3.39)
- removed the H3 at (39.7, -24.2)
- removed P1: Conn_01x01, Connector_Pin:Pin_D1.0mm_L10.0mm
- removed the Q4 at (5.94, -13.3)
- removed the Q5 at (5.94, -22.6)
- removed the Q6 at (1.89, -4.11)
- removed the Q7 at (17.5, -11.0)
- removed Q8, Q821, Q822, Q9: IRF830, valdiklio_footprints:TO-220-3_Vertical
- removed R805, R815, R825: 18k, Resistor_SMD:R_0805_2012Metric
- added C18: 1.0uFx50V, Capacitor_SMD:C_0805_2012Metric, F.Cu at (139.0, 131.2)
- added C2: 4.7x400V, Capacitor_THT:CP_Radial_D10.0mm_P5.00mm, F.Cu at (121.0, 44.0)
- added C20: 1.0uFx50V, Capacitor_SMD:C_0805_2012Metric, F.Cu at (83.2, 131.2)
- added C21: 0.1, Capacitor_SMD:C_0805_2012Metric, F.Cu at (136.7, 72.0)
- added C22: 0.1, Capacitor_SMD:C_0805_2012Metric, F.Cu at (142.2, 87.5)
- added C23: 0.1, Capacitor_SMD:C_0805_2012Metric, F.Cu at (139.5, 103.8)
- added C24: 1n0, Capacitor_SMD:C_0805_2012Metric, F.Cu at (190.7, 101.6)
- added C5: 4.7x400V, Capacitor_THT:CP_Radial_D10.0mm_P5.00mm, F.Cu at (133.0, 44.0)
- added C6: 1.0x50V, Capacitor_THT:CP_Radial_D5.0mm_P2.50mm, F.Cu at (154.8, 70.5)
- added D10: LL4148, Diode_SMD:D_MiniMELF, F.Cu at (155.2, 87.8)
- added D11: UF4005, Diode_THT:D_DO-41_SOD81_P7.62mm_Horizontal, F.Cu at (143.5, 130.2)
- added D12: UF4005, Diode_THT:D_DO-41_SOD81_P7.62mm_Horizontal, F.Cu at (115.5, 141.5)
- added D13: UF4005, Diode_THT:D_DO-41_SOD81_P7.62mm_Horizontal, F.Cu at (88.5, 130.2)
- added D14: LL4148, Diode_SMD:D_MiniMELF, F.Cu at (150.2, 123.5)
- added D17: LL4148, Diode_SMD:D_MiniMELF, F.Cu at (104.0, 137.6)
- added D18: LL4148, Diode_SMD:D_MiniMELF, F.Cu at (89.5, 136.2)
- added D19: LL4148, Diode_SMD:D_MiniMELF, F.Cu at (78.8, 133.4)
- added D2: LL4005, Diode_SMD:D_MELF, F.Cu at (110.0, 48.6)
- added D20: LL4148, Diode_SMD:D_MiniMELF, F.Cu at (190.7, 104.1)
- added D22: D, Diode_THT:D_DO-201AD_P15.24mm_Horizontal, F.Cu at (105.0, 52.8)
- added D23: D, Diode_THT:D_DO-201AD_P15.24mm_Horizontal, F.Cu at (99.0, 52.8)
- added D24: D, Diode_THT:D_DO-201AD_P15.24mm_Horizontal, F.Cu at (83.8, 68.0)
- added D25: D, Diode_THT:D_DO-201AD_P15.24mm_Horizontal, F.Cu at (89.5, 68.0)
- added D3: LL4005, Diode_SMD:D_MELF, F.Cu at (94.0, 48.6)
- added D4: LL4148, Diode_SMD:D_MiniMELF, F.Cu at (153.8, 62.8)
- added D5: UF4005, Diode_THT:D_DO-41_SOD81_P10.16mm_Horizontal, F.Cu at (111.0, 56.5)
- added D6: 12V, Diode_SMD:D_MiniMELF, F.Cu at (127.8, 65.2)
- added D7: LL4148, Diode_SMD:D_MiniMELF, F.Cu at (166.5, 65.0)
- added D8: LL4148, Diode_SMD:D_MiniMELF, F.Cu at (155.2, 85.5)
- added D9: LL4148, Diode_SMD:D_MiniMELF, F.Cu at (155.2, 83.2)
- added F1: 3A, Fuse:Fuseholder_TR5_Littelfuse_No560_No460, F.Cu at (85.8, 37.8)
- added F2: 5A, Fuse:Fuseholder_TR5_Littelfuse_No560_No460, F.Cu at (76.0, 43.3)
- added L1: 1mH, Inductor_SMD:L_Vishay_IHSM-3825, F.Cu at (126.2, 51.0)
- added L2: 1mH/280mA, Inductor_THT:L_Radial_D7.8mm_P5.00mm_Fastron_07HCP, F.Cu at (118.8, 56.5)
- added Q1: BC807, Package_TO_SOT_SMD:SOT-23, F.Cu at (159.5, 64.5)
- added Q2: IRF830, valdiklio_footprints:TO-220-3_Vertical, F.Cu at (153.0, 130.0)
- added Q3: IRF830, valdiklio_footprints:TO-220-3_Vertical, F.Cu at (139.0, 141.0)
- added R1: 1k, Resistor_SMD:R_0805_2012Metric, F.Cu at (138.8, 33.2)
- added R19: 1k0, Resistor_SMD:R_0805_2012Metric, F.Cu at (152.6, 92.0)
- added R2: 1k0, Resistor_SMD:R_0805_2012Metric, F.Cu at (233.2, 52.9)
- added R21: 1k0, Resistor_SMD:R_0805_2012Metric, F.Cu at (152.6, 94.0)
- added R22: 47R, Resistor_SMD:R_0805_2012Metric, F.Cu at (146.8, 122.8)
- added R23: 47R, Resistor_SMD:R_0805_2012Metric, F.Cu at (131.7, 131.0)
- added R24: 47R, Resistor_SMD:R_0805_2012Metric, F.Cu at (118.5, 137.2)
- added R25: 47R, Resistor_SMD:R_0805_2012Metric, F.Cu at (100.2, 137.6)
- added R26: 47R, Resistor_SMD:R_0805_2012Metric, F.Cu at (92.8, 136.1)
- added R27: 47R, Resistor_SMD:R_0805_2012Metric, F.Cu at (75.0, 133.4)
- added R28: 1K0, Resistor_SMD:R_0805_2012Metric, F.Cu at (152.4, 133.3)
- added R29: 1K0, Resistor_SMD:R_0805_2012Metric, F.Cu at (119.3, 149.9)
- added R3: 10k, Resistor_SMD:R_0805_2012Metric, F.Cu at (234.5, 56.7)
- added R30: 1K0, Resistor_SMD:R_0805_2012Metric, F.Cu at (81.2, 143.5)
- added R31: 1K0, Resistor_SMD:R_0805_2012Metric, F.Cu at (137.4, 144.2)
- added R32: 1K0, Resistor_SMD:R_0805_2012Metric, F.Cu at (99.6, 150.1)
- added R33: 1K0, Resistor_SMD:R_0805_2012Metric, F.Cu at (66.6, 132.6)
- added R34: 0R1, Resistor_THT:R_Axial_DIN0309_L9.0mm_D3.2mm_P12.70mm_Horizontal, F.Cu at (202.0, 106.2)
- added R38: 1K0, Resistor_SMD:R_0805_2012Metric, F.Cu at (194.5, 99.1)
- added R39: 1K0, Resistor_SMD:R_0805_2012Metric, F.Cu at (190.7, 99.1)
- added R4: 8R2/2W, Resistor_THT:R_Axial_DIN0411_L9.9mm_D3.6mm_P12.70mm_Horizontal, F.Cu at (90.3, 42.0)
- added R40: 220k, Resistor_THT:R_Axial_DIN0411_L9.9mm_D3.6mm_P12.70mm_Horizontal, F.Cu at (95.2, 73.2)
- added R5: 10k, Resistor_SMD:R_0805_2012Metric, F.Cu at (239.5, 55.4)
- added R6: 490, Resistor_SMD:R_0805_2012Metric, F.Cu at (153.8, 58.3)
- added RV1: Varistor, Varistor:RV_Disc_D9mm_W4mm_P5mm, F.Cu at (84.0, 46.1)
- added RV2: Varistor, Varistor:RV_Disc_D9mm_W4mm_P5mm, F.Cu at (104.0, 48.0)
- added TH1: 33R, Varistor:RV_Disc_D9mm_W4mm_P5mm, F.Cu at (100.0, 38.0)
- added U10: IR2101, Package_SO:SOIC-8_3.9x4.9mm_P1.27mm, F.Cu at (82.8, 126.2)
- added U2: CNY17-1, Package_DIP:DIP-6_W7.62mm, F.Cu at (230.7, 38.9)
- added U3: CNY17-1, Package_DIP:DIP-6_W7.62mm, F.Cu at (233.2, 64.3)
- added U4: LNK304G, Package_DIP:PowerIntegrations_SMD-8B, F.Cu at (144.8, 49.2)
- added U7: STM32F103C8Tx, Package_QFP:LQFP-48_7x7mm_P0.5mm, F.Cu at (164.5, 83.2)
- added U8: IR2101, Package_SO:SOIC-8_3.9x4.9mm_P1.27mm, F.Cu at (138.2, 126.2)
- added U9: IR2101, Package_SO:SOIC-8_3.9x4.9mm_P1.27mm, F.Cu at (110.0, 137.5)
- added VP1: R_POT_TRIM, Potentiometer_THT:Potentiometer_ACP_CA6-H2,5_Horizontal, F.Cu at (141.0, 36.0)
- C1: renamed from C102; value 120.0x400V -> 120x400V
- C10, C11, C12: value 1.0uFx50V -> 100n
- C13: value 0.1 -> 100x16V; footprint Capacitor_SMD:C_0805_2012Metric -> Capacitor_THT:CP_Radial_D6.3mm_P2.50mm
- C14, C15: value 0.1 -> 100n
- C16, C17: value 4.7x400V -> 100n; footprint Capacitor_THT:C_Radial_D10.0mm_H20.0mm_P5.00mm -> Capacitor_SMD:C_0805_2012Metric
- C19: value 100x16V -> 1.0uFx50V; footprint Capacitor_THT:C_Radial_D6.3mm_H5.0mm_P2.50mm -> Capacitor_SMD:C_0805_2012Metric
- C3: renamed from C101; value 120.0x400V -> 120x400V
- C4: renamed from C100; value 120.0x400V -> 120x400V
- C7, C9: value C -> 100n
- C8: value C -> 100x16V; footprint Capacitor_SMD:C_0805_2012Metric -> Capacitor_THT:CP_Radial_D6.3mm_P2.50mm
- D15, D16: value LL4005 -> LL4148; footprint Diode_SMD:D_MELF -> Diode_SMD:D_MiniMELF
- H1: renamed from H600; value HALL -> SA
- H2: renamed from H601; value HALL -> SB
- H3: renamed from H602; value HALL -> SC
- J3: value HALLS -> ISP_SWD_Connector; footprint Connector_PinHeader_2.54mm:PinHeader_1x05_P2.54mm_Vertical -> mech:ISP_SWD_Connector
- R10: value R -> 1M
- R11: value R -> 2.2k
- R12: value R -> 33k
- R13: value 1K0 -> 22k
- R14: value 1K0 -> 4k7
- R15, R17: value 1K0 -> 10k
- R16: value 1K0 -> 100k
- R20, R9: value R -> 1k0
- R7: value R -> 20k
- R8: value R -> 10k
- U1: value STM32F103C8Tx -> CNY17-1; footprint Package_QFP:LQFP-48_7x7mm_P0.5mm -> Package_DIP:DIP-6_W7.62mm
- U5: value LNK304G -> PC817; footprint Package_DIP:PowerIntegrations_SMD-8B -> Package_DIP:DIP-4_W10.16mm_LongPads
- U6: value PC817 -> SIP21106; footprint Package_DIP:DIP-4_W7.62mm -> Package_TO_SOT_SMD:SOT-23-5
- moved J3 204.7 mm to (168.0, 74.8), turned to 90 degrees
- moved R9 201.4 mm to (229.4, 60.5)
- moved C10 187.8 mm to (162.8, 67.7), turned to 90 degrees
- moved C16 179.4 mm to (112.0, 131.8), turned to 270 degrees
- moved D15 177.1 mm to (134.2, 131.0), turned to 270 degrees
- moved C19 176.5 mm to (110.8, 142.5)
- moved D16 168.5 mm to (122.3, 137.2), turned to 270 degrees
- moved U6 168.1 mm to (146.0, 59.8)
- moved C17 167.7 mm to (84.8, 120.6), turned to 270 degrees
- moved R18 164.2 mm to (162.3, 99.8)
- moved C15 164.2 mm to (140.2, 120.5), turned to 270 degrees
- moved C14 163.8 mm to (162.3, 97.8)
- moved C7 156.2 mm to (138.0, 55.2), turned to 270 degrees
- moved U5 149.6 mm to (127.8, 58.2)
- moved R20 148.7 mm to (152.6, 90.0)
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- renumbered Q811 to Q4, Q812 to Q5, Q801 to Q6, Q802 to Q7
Connections:
- net /+V renamed /VB
- net /PE renamed Net-(J1-Pad3)
- C1 pad 2: Net-(C100-Pad2) -> GND
- C10 pad 1: /PHA -> GND
- C10 pad 2: Net-(C10-Pad2) -> /~NRST
- C11 pad 1: /PHB -> GND
- C12 pad 1: /PHC -> GND
- C12 pad 2: Net-(C12-Pad2) -> /3VDC
- C13 pad 1: GND -> /3VDC
- C13 pad 2: /VCC -> GND
- C14 pad 2: /VCC -> /TEMP
- C16 pad 1: Net-(C16-Pad1) -> GND
- C16 pad 2: Net-(C16-Pad2) -> /VCC
- C17 pad 1: Net-(C17-Pad1) -> GND
- C17 pad 2: Net-(C16-Pad2) -> /VCC
- C19 pad 1: Net-(C19-Pad1) -> /PHB
- C19 pad 2: Net-(C16-Pad2) -> Net-(C19-Pad2)
- C3 pad 2: Net-(C100-Pad2) -> GND
- C4 pad 2: Net-(C100-Pad2) -> GND
- C7 pad 1: GND -> Net-(C7-Pad1)
- C7 pad 2: /VCC -> Net-(C7-Pad2)
- C8 pad 1: GND -> /VCC
- C8 pad 2: /VCC -> GND
- D15 pad 1: Net-(C16-Pad1) -> Net-(D15-Pad1)
- D16 pad 2: Net-(C16-Pad2) -> Net-(D16-Pad2)
- H1 pad 2: Net-(H600-Pad2) -> Net-(H1-Pad2)
- J1 pad 1: Net-(F1-Pad2) -> /ACL
- J1 pad 2: Net-(D100-Pad2) -> /ACN
- J1 pad 4: /OKP -> /OKM
- J1 pad 5: /OKM -> /OKP
- J3 pad 1: /VCC -> /SWDIO
- J3 pad 2: /~SA -> GND
- J3 pad 3: /~SB -> /SWDCLK
- J3 pad 4: /~SC -> /~NRST
- J3 pad 5: GND -> /3VDC
- Q4 pad 1: Net-(Q811-Pad1) -> Net-(D16-Pad2)
- Q4 pad 2: /+U -> Net-(Q4-Pad2)
- Q4 pad 3: Net-(P2-Pad1) -> /PHB
- Q5 pad 2: Net-(P2-Pad1) -> /PHB
- Q6 pad 2: /+U -> Net-(Q6-Pad2)
- Q6 pad 3: Net-(P1-Pad1) -> /PHC
- Q7 pad 2: Net-(P1-Pad1) -> /PHC
- R10 pad 1: Net-(D12-Pad2) -> Net-(Q1-Pad2)
- R10 pad 2: Net-(D12-Pad1) -> Net-(Q1-Pad1)
- R11 pad 1: Net-(D13-Pad2) -> Net-(Q1-Pad3)
- R11 pad 2: Net-(D13-Pad1) -> GND
- R12 pad 1: Net-(D14-Pad2) -> /SPEED
- R12 pad 2: Net-(D14-Pad1) -> Net-(Q1-Pad3)
- R13 pad 1: /PHA -> /SPEED
- R13 pad 2: Net-(D9-Pad2) -> GND
- R14 pad 1: /PHB -> Net-(D6-Pad1)
- R14 pad 2: Net-(D11-Pad2) -> /VCC
- R15 pad 1: /PHC -> /VCC
- R15 pad 2: Net-(D13-Pad2) -> Net-(R15-Pad2)
- R16 pad 1: Net-(Q5-Pad3) -> Net-(R16-Pad1)
- R16 pad 2: Net-(D10-Pad2) -> GND
- R17 pad 1: Net-(Q5-Pad3) -> /3VDC
- R17 pad 2: Net-(D12-Pad2) -> /~NRST
- R18 pad 1: Net-(Q5-Pad3) -> GND
- R18 pad 2: Net-(D14-Pad2) -> /TEMP
- R20 pad 1: Net-(D18-Pad1) -> Net-(H1-Pad2)
- R20 pad 2: Net-(C19-Pad1) -> /SA
- R7 pad 1: Net-(D9-Pad2) -> Net-(D4-Pad1)
- R7 pad 2: Net-(D9-Pad1) -> Net-(Q1-Pad1)
- R8 pad 1: Net-(D10-Pad2) -> Net-(Q1-Pad1)
- R8 pad 2: Net-(D10-Pad1) -> GND
- R9 pad 1: Net-(D11-Pad2) -> /TXD
- U1 pad 2: /LED -> /OKM
- U1 pad 4: Net-(U1-Pad4) -> Net-(Q1-Pad2)
- U5 pad 1: Net-(C18-Pad1) -> /VCC
- U5 pad 2: Net-(C18-Pad1) -> Net-(D6-Pad1)
- U5 pad 3: Net-(C18-Pad2) -> Net-(U4-Pad4)
- U5 pad 4: Net-(U5-Pad4) -> Net-(C7-Pad2)
- U6 pad 1: Net-(C19-Pad1) -> /VCC
- U6 pad 2: Net-(D18-Pad1) -> GND
- U6 pad 3: Net-(U5-Pad4) -> Net-(R15-Pad2)
- U6 pad 4: Net-(C18-Pad2) -> Net-(C11-Pad2)

Commit message: plokstes testavimams
Parts:
- removed the D8 at (155.2, 85.5)
- removed the D9 at (155.2, 83.2)
- removed Q2: IRF830, valdiklio_footprints:TO-220-3_Vertical
- removed the R19 at (152.6, 92.0)
- removed the R20 at (152.6, 90.0)
- removed the R21 at (152.6, 94.0)
- added C12: 100x16V, Capacitor_THT:CP_Radial_D6.3mm_P2.50mm, F.Cu at (149.0, 72.5)
- added C13: 100n, Capacitor_SMD:C_0805_2012Metric, F.Cu at (144.0, 67.6)
- added C20: 1n0, Capacitor_SMD:C_0805_2012Metric, F.Cu at (168.4, 10.9)
- added C25: 1n0, Capacitor_SMD:C_0805_2012Metric, F.Cu at (154.4, 2.06)
- added C7: 100n, Capacitor_SMD:C_0805_2012Metric, F.Cu at (98.3, 2.52)
- added D12: LL4148, Diode_SMD:D_MiniMELF, F.Cu at (119.2, -0.25)
- added D15: LL4148, Diode_SMD:D_MiniMELF, F.Cu at (155.2, 145.6)
- added D16: LL4148, Diode_SMD:D_MiniMELF, F.Cu at (124.0, 159.5)
- added D17: LL4148, Diode_SMD:D_MiniMELF, F.Cu at (75.7, 151.9)
- added D18: LL4148, Diode_SMD:D_MiniMELF, F.Cu at (168.1, 5.09)
- added K1: Omron, Relay_THT:Relay_SPDT_Finder_34.51_Vertical, F.Cu at (16.0, 56.6)
- added Q4: IRF830, valdiklio_footprints:TO-220-3_Vertical, F.Cu at (139.0, 141.0)
- added R10: 100k, Resistor_SMD:R_1206_3216Metric, F.Cu at (93.3, -0.60)
- added R12: 100k, Resistor_SMD:R_1206_3216Metric, F.Cu at (93.3, 2.69)
- added R14: 100k, Resistor_SMD:R_1206_3216Metric, F.Cu at (98.9, -0.60)
- added R16: 2k2, Resistor_SMD:R_0805_2012Metric, F.Cu at (102.7, 2.52)
- added R25: 10k, Resistor_SMD:R_0805_2012Metric, F.Cu at (173.2, 8.41)
- added R33: 30R, Resistor_SMD:R_0805_2012Metric, F.Cu at (149.4, 149.4)
- added R34: 30R, Resistor_SMD:R_0805_2012Metric, F.Cu at (101.1, 163.3)
- added R35: 30R, Resistor_SMD:R_0805_2012Metric, F.Cu at (83.3, 155.7)
- added RN1: 1k0, Resistor_SMD:R_Array_Convex_4x0603, F.Cu at (155.0, 95.2)
- added U12: ACS712, Package_SO:SOIC-8_3.9x4.9mm_P1.27mm, F.Cu at (160.7, 6.69)
- added U6: LM340MP-5.0, disc:LM340_SOT-223, F.Cu at (146.8, 61.8)
- D19: renamed from D11; value UF4005 -> LL4005
- D20: renamed from D12; value UF4005 -> LL4005
- D21: renamed from D13; value UF4005 -> LL4005
- R26: renamed from R38; value 1K0 -> 2k0
- moved D10 144.0 mm to (13.4, 62.8)
- moved Q3 17.8 mm to (153.0, 130.0), turned to 225 degrees
- moved C16 11.9 mm to (157.2, 72.8), turned to 270 degrees
- moved C11 10.5 mm to (165.3, 77.8)
- moved D11 10.5 mm to (169.0, 75.2)
- moved J2 10.5 mm to (170.5, 84.9)
- moved R19 10.5 mm to (164.8, 85.2)
- moved R20 10.5 mm to (165.3, 74.3)
- moved C16 10.2 mm to (162.3, 107.9)
- moved R19 10.2 mm to (162.3, 109.9)
- moved U7 10.2 mm to (164.5, 93.4)
- moved R13 9.92 mm to (167.1, 61.6)
- moved R15 9.92 mm to (165.1, 61.6)
- moved R17 9.92 mm to (166.2, 64.2)
- moved U8 8.54 mm to (149.0, 67.8)
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- renumbered C9 to C10, C10 to C11, C11 to C14, C12 to C15, C14 to C16, C13 to C16, C15 to C17, C16 to C18, C17 to C19, C18 to C21, C19 to C22, C20 to C23, C21 to C26, C22 to C27, C23 to C28, C5 to C4, C4 to C5, C7 to C8, C8 to C9, D22 to D1, D7 to D11, D23 to D2, D14 to D22, D15 to D23, D16 to D24, D17 to D25, D18 to D26, D19 to D27, D24 to D3, D25 to D4, D2 to D5, D3 to D6, D4 to D7, D5 to D8, D6 to D9, F2 to F1, F1 to F2, J3 to J2, Q4 to Q5, Q5 to Q6, Q6 to Q7, Q7 to Q8, R10 to R11, R11 to R13, R12 to R15, R13 to R17, R14 to R18, R16 to R19, R18 to R19, R17 to R20, R15 to R21, R22 to R27, R23 to R28, R24 to R29, R25 to R30, R26 to R31, R28 to R31, R27 to R32, R29 to R32, R30 to R33, R31 to R34, R32 to R35, R33 to R36, R40 to R5, RV2 to RV1, RV1 to RV2, U9 to U10, U10 to U11, U6 to U8, U8 to U9
Connections:
- net /~CHA renamed /CHAN
- net /~CHB renamed /CHBN
- net /~CHC renamed /CHCN
- net Net-(U7-Pad20) renamed /VBON
- net Net-(U7-Pad3) renamed /DIR
- net Net-(U7-Pad4) renamed /TEMPON
- C1 pad 1: /VB -> Net-(C1-Pad1)
- C1 pad 2: GND -> GNDD
- C10 pad 1: GND -> GNDD
- C11 pad 1: GND -> GNDD
- C14 pad 1: GND -> GNDD
- C15 pad 1: GND -> GNDD
- C16 pad 2: GND -> GNDD
- C17 pad 1: GND -> GNDD
- C18 pad 1: GND -> GNDD
- C19 pad 1: GND -> GNDD
- C2 pad 2: GND -> GNDD
- C21 pad 1: /PHA -> Net-(C21-Pad1)
- C21 pad 2: Net-(C18-Pad2) -> Net-(C21-Pad2)
- C22 pad 1: /PHB -> Net-(C22-Pad1)
- C22 pad 2: Net-(C19-Pad2) -> Net-(C22-Pad2)
- C23 pad 1: /PHC -> Net-(C23-Pad1)
- C23 pad 2: Net-(C20-Pad2) -> Net-(C23-Pad2)
- C24 pad 1: GND -> GNDD
- C24 pad 2: /CURR -> Net-(C24-Pad2)
- C26 pad 1: GND -> GNDD
- C27 pad 1: GND -> GNDD
- C28 pad 1: GND -> GNDD
- C3 pad 1: /VB -> Net-(C1-Pad1)
- C3 pad 2: GND -> GNDD
- C4 pad 2: GND -> GNDD
- C5 pad 1: /VB -> Net-(C1-Pad1)
- C5 pad 2: GND -> GNDD
- C6 pad 2: GND -> GNDD
- C9 pad 2: GND -> GNDD
- D1 pad 2: GND -> GNDD
- D10 pad 1: /3VDC -> /VCC
- D10 pad 2: /SC -> Net-(D10-Pad2)
- D19 pad 1: Net-(C18-Pad2) -> Net-(C21-Pad1)
- D19 pad 2: /VCC -> GNDD
- D2 pad 2: GND -> GNDD
- D20 pad 1: Net-(C19-Pad2) -> Net-(C22-Pad1)
- D20 pad 2: /VCC -> GNDD
- D21 pad 1: Net-(C20-Pad2) -> Net-(C23-Pad1)
- D21 pad 2: /VCC -> GNDD
- D22 pad 2: Net-(D14-Pad2) -> Net-(D22-Pad2)
- D23 pad 2: Net-(D15-Pad2) -> Net-(D23-Pad2)
- D24 pad 2: Net-(D16-Pad2) -> Net-(D24-Pad2)
- D25 pad 2: Net-(D17-Pad2) -> Net-(D25-Pad2)
- D26 pad 2: Net-(D18-Pad2) -> Net-(D26-Pad2)
- D27 pad 2: Net-(D19-Pad2) -> Net-(D27-Pad2)
- D3 pad 1: /VB -> Net-(C1-Pad1)
- D4 pad 1: /VB -> Net-(C1-Pad1)
- D6 pad 2: GND -> GNDD
- D8 pad 2: GND -> GNDD
- D9 pad 2: GND -> GNDD
- H1 pad 2: Net-(H1-Pad2) -> /SA
- H1 pad 3: GND -> GNDD
- H2 pad 2: Net-(H2-Pad2) -> /SB
- H2 pad 3: GND -> GNDD
- H3 pad 2: Net-(H3-Pad2) -> /SC
- H3 pad 3: GND -> GNDD
- J2 pad 2: GND -> GNDD
- J2 pad 6: GND -> GNDD
- Q3 pad 1: Net-(D15-Pad2) -> Net-(D22-Pad2)
- Q3 pad 2: /PHA -> /VB
- Q3 pad 3: Net-(Q3-Pad3) -> /PHA
- Q5 pad 1: Net-(D16-Pad2) -> Net-(D24-Pad2)
- Q5 pad 2: Net-(Q4-Pad2) -> /VB
- Q6 pad 1: Net-(D17-Pad2) -> Net-(D25-Pad2)
- Q6 pad 3: Net-(Q3-Pad3) -> Net-(Q4-Pad3)
- Q7 pad 1: Net-(D18-Pad2) -> Net-(D26-Pad2)
- Q7 pad 2: Net-(Q6-Pad2) -> /VB
- Q8 pad 1: Net-(D19-Pad2) -> Net-(D27-Pad2)
- Q8 pad 3: Net-(Q3-Pad3) -> Net-(Q4-Pad3)
- R13 pad 2: GND -> GNDD
- R17 pad 2: GND -> GNDD
- R19 pad 2: GND -> GNDD
- R21 pad 1: /VCC -> /5VDC
- R26 pad 1: /CURR -> Net-(R26-Pad1)
- R26 pad 2: Net-(Q3-Pad3) -> Net-(D18-Pad2)
- R27 pad 1: Net-(D14-Pad2) -> Net-(D22-Pad2)
- R28 pad 1: Net-(D15-Pad2) -> Net-(D23-Pad2)
- R29 pad 1: Net-(D16-Pad2) -> Net-(D24-Pad2)
- R3 pad 2: GNDD -> GND
- R30 pad 1: Net-(D17-Pad2) -> Net-(D25-Pad2)
- R31 pad 1: Net-(D18-Pad2) -> Net-(D26-Pad2)
- R31 pad 2: Net-(D14-Pad2) -> Net-(D18-Pad2)
- R32 pad 1: Net-(D19-Pad2) -> Net-(D27-Pad2)
- R32 pad 2: Net-(D16-Pad2) -> Net-(D20-Pad2)
- R33 pad 2: Net-(D18-Pad2) -> Net-(D22-Pad2)
- R34 pad 2: Net-(D15-Pad2) -> Net-(D19-Pad2)
- R35 pad 2: Net-(D17-Pad2) -> Net-(D21-Pad2)
- R36 pad 2: Net-(D19-Pad2) -> Net-(D23-Pad2)
- R5 pad 2: GND -> GNDD
- R5 pad 2: /VB -> Net-(C1-Pad1)
- R8 pad 2: GND -> GNDD
- U10 pad 4: GND -> GNDD
- U10 pad 6: /PHB -> Net-(C22-Pad1)
- U10 pad 8: Net-(C19-Pad2) -> Net-(C22-Pad2)
- U11 pad 4: GND -> GNDD
- U11 pad 6: /PHC -> Net-(C23-Pad1)
- U11 pad 8: Net-(C20-Pad2) -> Net-(C23-Pad2)
- U2 pad 2: GNDD -> GND
- U3 pad 2: GND -> GNDD
- U7 pad 23: GND -> GNDD
- U7 pad 35: GND -> GNDD
- U7 pad 47: GND -> GNDD
- U7 pad 8: GND -> GNDD
- U8 pad 1: /VCC -> /5VDC
- U8 pad 2: GND -> GNDD
- U9 pad 4: GND -> GNDD
- U9 pad 6: /PHA -> Net-(C21-Pad1)
- U9 pad 8: Net-(C18-Pad2) -> Net-(C21-Pad2)
